File: cellboard/CellsBoard.sch (KiCad schematic (older format))
At the start: 38 parts, among them U15 CellBoardConnection

Commit message: removed rescue references and rescue library
Parts:
- JP1, JP10, JP11, JP12, JP13, JP14, JP15, JP16, JP17, JP18, JP2, JP3, JP4, JP5, JP6, JP7, JP8, JP9: symbol Device:Jumper_NC_Small -> CellsBoard:Jumper_NC_Small
Changed lines of the file:
@@
 $EndComp
 $Comp
-L Device:Jumper_NC_Small JP15
+L CellsBoard:Jumper_NC_Small JP15
 U 1 1 5E68F5DB
 P 7050 2150
@@
 $EndComp
 $Comp
-L Device:Jumper_NC_Small JP16
+L CellsBoard:Jumper_NC_Small JP16
 U 1 1 5E68F5E1
 P 7050 2050
@@
 $EndComp
 $Comp
-L Device:Jumper_NC_Small JP13
+L CellsBoard:Jumper_NC_Small JP13
 U 1 1 5E68F5E7
 P 7050 2350
@@
 $EndComp
 $Comp
-L Device:Jumper_NC_Small JP14
+L CellsBoard:Jumper_NC_Small JP14
 U 1 1 5E68F5ED
 P 7050 2250
@@
 $EndComp
 $Comp
-L Device:Jumper_NC_Small JP17
+L CellsBoard:Jumper_NC_Small JP17
 U 1 1 5E68F5F3
 P 7050 1950
@@
 $EndComp
 $Comp
-L Device:Jumper_NC_Small JP18
+L CellsBoard:Jumper_NC_Small JP18
 U 1 1 5E68F5F9
 P 7050 1850
@@
 $EndComp
 $Comp
-L Device:Jumper_NC_Small JP9
+L CellsBoard:Jumper_NC_Small JP9
 U 1 1 5E69CC76
 P 7050 2750
@@
 $EndComp
 $Comp
-L Device:Jumper_NC_Small JP10
+L CellsBoard:Jumper_NC_Small JP10
 U 1 1 5E69CC7C
 P 7050 2650
@@
 $EndComp
 $Comp
-L Device:Jumper_NC_Small JP7
+L CellsBoard:Jumper_NC_Small JP7
 U 1 1 5E69CC82
 P 7050 2950
@@
 $EndComp
 $Comp
-L Device:Jumper_NC_Small JP8
+L CellsBoard:Jumper_NC_Small JP8
 U 1 1 5E69CC88
 P 7050 2850
@@
 $EndComp
 $Comp
-L Device:Jumper_NC_Small JP11
+L CellsBoard:Jumper_NC_Small JP11
 U 1 1 5E69CC8E
 P 7050 2550
@@
 $EndComp
 $Comp
-L Device:Jumper_NC_Small JP12
+L CellsBoard:Jumper_NC_Small JP12
 U 1 1 5E69CC94
 P 7050 2450
@@
 $EndComp
 $Comp
-L Device:Jumper_NC_Small JP3
+L CellsBoard:Jumper_NC_Small JP3
 U 1 1 5E6A3AFC
 P 7050 3350
@@
 $EndComp
 $Comp
-L Device:Jumper_NC_Small JP4
+L CellsBoard:Jumper_NC_Small JP4
 U 1 1 5E6A3B02
 P 7050 3250
@@
 $EndComp
 $Comp
-L Device:Jumper_NC_Small JP1
+L CellsBoard:Jumper_NC_Small JP1
 U 1 1 5E6A3B08
 P 7050 3550
@@
 $EndComp
 $Comp
-L Device:Jumper_NC_Small JP2
+L CellsBoard:Jumper_NC_Small JP2
 U 1 1 5E6A3B0E
 P 7050 3450
@@
 $EndComp
 $Comp
-L Device:Jumper_NC_Small JP5
+L CellsBoard:Jumper_NC_Small JP5
 U 1 1 5E6A3B14
 P 7050 3150
@@
 $EndComp
 $Comp
-L Device:Jumper_NC_Small JP6
+L CellsBoard:Jumper_NC_Small JP6
 U 1 1 5E6A3B1A
 P 7050 3050
