File: cellboard/CellsBoard.sch (KiCad schematic (older format))
At the start: 38 parts, among them U15 CellBoardConnection

Commit message: v2.1.2.5 as printed
Commit on behalf of fran-retfie.
Parts:
- removed JP1, JP10, JP11, JP12, JP13, JP14, JP15, JP16, JP17, JP18, JP2, JP3, JP4, JP5, JP6, JP7, JP8, JP9: Jumper_NC_Small, CellsBoard:JUMPER_NC, symbol CellsBoard:Jumper_NC_Small
- removed U15: CellBoardConnection, CellsBoard:CELL_SPACE_FINAL, symbol CellsBoard:CellBoardConnection
- added F20, F21, F22, F23, F24, F25: Fuse, CellsBoard:Fuse_0805, symbol Device:Fuse
- added J1, J2, J3, J4, J5, J6: Conn_02x02_Odd_Even, Connector_Molex:Molex_Micro-Fit_3.0_43045-0412_2x02_P3.00mm_Vertical, symbol Connector_Generic:Conn_02x02_Odd_Even
- added NT0, NT1, NT10, NT11, NT12, NT13, NT14, NT15, NT16, NT17, NT18, NT19, NT2, NT3, NT4, NT5, NT6, NT7, NT8, NT9: Net-Tie_2, NetTie:NetTie-2_SMD_Pad0.5mm, symbol Device:Net-Tie_2
- added NT20: Net-Tie_2, NetTie:NetTie-2_SMD_Pad2.0mm, symbol Device:Net-Tie_2
- added TP1, TP2, TP3, TP4, TP7: TestPoint, CellsBoard:TestPoint_GNDedge_toponly, symbol Connector:TestPoint
- added TP12: VCC, TestPoint:TestPoint_Pad_D1.0mm, symbol Connector:TestPoint
- F1, F10, F11, F12, F13, F14, F15, F16, F17, F18, F19, F2, F3, F4, F5, F6, F7, F8, F9: symbol CellsBoard:Fuse -> Device:Fuse
Connections:
- net BATTERY MANAGER/CB1: now also NT1.2
- net BATTERY MANAGER/CB10: now also NT10.2
- net BATTERY MANAGER/CB11: now also NT11.2
- net BATTERY MANAGER/CB12: now also NT12.2
- net BATTERY MANAGER/CB13: now also NT13.2
- net BATTERY MANAGER/CB14: now also NT14.2
- net BATTERY MANAGER/CB15: now also NT15.2
- net BATTERY MANAGER/CB16: now also NT16.2
- net BATTERY MANAGER/CB17: now also NT17.2
- net BATTERY MANAGER/CB18: now also NT18.2
- net BATTERY MANAGER/CB2: now also NT2.2
- net BATTERY MANAGER/CB3: now also NT3.2
- net BATTERY MANAGER/CB4: now also NT4.2
- net BATTERY MANAGER/CB5: now also NT5.2
- net BATTERY MANAGER/CB6: now also NT6.2
- net BATTERY MANAGER/CB7: now also NT7.2
- net BATTERY MANAGER/CB8: now also NT8.2
- net BATTERY MANAGER/CB9: now also NT9.2
- net CB0N: now also J6.4 (Pin_4), NT19.1
- net CB1: now also NT1.1
- net CB10: now also NT10.1
- net CB10N: now also J3.2 (Pin_2)
- net CB11: now also NT11.1
- net CB11N: now also J3.1 (Pin_1)
- net CB12: now also F21.2, NT12.1
- net CB13: now also NT13.1
- net CB13N: now also J2.2 (Pin_2)
- net CB14: now also NT14.1
- net CB14N: now also J2.1 (Pin_1)
- net CB15: now also F20.2, NT15.1
- net CB16: now also NT16.1
- net CB16N: now also J1.2 (Pin_2)
- net CB17: now also NT17.1
- net CB17N: now also J1.1 (Pin_1)
- net CB18: now also NT18.1
- net CB18N: now also F25.1, J1.3 (Pin_3)
- net CB1N: now also J6.2 (Pin_2)
- net CB2: now also NT2.1
- net CB2N: now also J6.1 (Pin_1)
- net CB3: now also F24.2, NT3.1
- net CB4: now also NT4.1
- net CB4N: now also J5.2 (Pin_2)
- net CB5: now also NT5.1
- net CB5N: now also J5.1 (Pin_1)
- net CB6: now also F23.2, NT6.1
- net CB7: now also NT7.1
- net CB7N: now also J4.2 (Pin_2)
- net CB8: now also NT8.1
- net CB8N: now also J4.1 (Pin_1)
- net CB9: now also F22.2, NT9.1
- net GND: now also NT19.2, NT20.2, TP1.1, TP2.1, TP3.1, TP4.1; no longer F1.2
- net CB12N renamed CB12N-1
- net CB12N-1: now also J2.4 (Pin_4)
- net CB15N renamed CB15N-1
- net CB15N-1: now also J1.4 (Pin_4)
- net CB3N renamed CB3N-1
- net CB3N-1: now also J5.4 (Pin_4)
- net CB6N renamed CB6N-1
- net CB6N-1: now also J4.4 (Pin_4)
- net CB9N renamed CB9N-2
- net CB9N-2: now also J3.4 (Pin_4)
- new net BATTERY MANAGER/CB0: NT0.2
- new net CB0: F1.2, NT0.1
- new net CB12N-2: F21.1, J3.3 (Pin_3)
- new net CB15N-2: F20.1, J2.3 (Pin_3)
- new net CB3N-2: F24.1, J6.3 (Pin_3)
- new net CB6N-2: F23.1, J5.3 (Pin_3)
- new net CB9N-1: F22.1, J4.3 (Pin_3)
- new net DCDC_80Vto5V/GND_SUPPLY: NT20.1, TP7.1
- new net VCC: F25.2, TP12.1
Other:
- note added: "POWER"
- note added: "SENSE"
- moved on the sheet: F1, F10, F11, F12, F13, F14, F15, F16, F17, F18, F19, F2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
