File: cellboard/Temperature section.sch (KiCad schematic (older format))
At the start: 26 parts, among them J10 BUS, J7 CONN_1x08, J9 BUS, SW1 RESET, U10 M95256-W, U11 MAX14878AWA+, U2 MCP1812, U5 STM32G474CxU

Commit message: removed rescue references and rescue library
Parts:
- U10: symbol CellsBoard-rescue:M95M56-WMN6P-Memory_EEPROM -> Memory_EEPROM:M95256-WMN6P
Changed lines of the file:
@@
 	5900 5000 5500 5000
 $Comp
-L CellsBoard-rescue:M95M56-WMN6P-Memory_EEPROM U10
+L Memory_EEPROM:M95256-WMN6P U10
 U 1 1 5E6762DB
 P 7200 1300
