File: cellboard/Balance.sch (KiCad schematic (older format))
At the start: 59 parts, among them Q1 BSS308PE, Q10 BSS308PE, Q11 BSS308PE, Q12 BSS308PE, Q13 BSS308PE, Q14 BSS308PE, Q15 BSS308PE, Q16 BSS308PE, Q17 BSS308PE, Q18 BSS308PE, Q2 BSS308PE, Q3 BSS308PE, Q4 BSS308PE, Q5 BSS308PE, Q6 BSS308PE, Q7 BSS308PE, Q8 BSS308PE, Q9 BSS308PE

Commit message: v2.1.2.5 as printed
Commit on behalf of fran-retfie.
Parts:
- removed R1, R10, R11, R12, R13, R14, R15, R16, R17, R18, R2, R3, R4, R5, R6, R7, R8, R9: Rdsc, Resistor_SMD:R_2512_6332Metric, symbol CellsBoard:R
- Q1, Q10, Q11, Q12, Q13, Q14, Q2, Q3, Q4, Q5, Q6, Q7, Q8, Q9: value BSS308PE -> TSM3401CX RFG
- R32, R33, R34, R35, R36, R37, R38, R39, R40, R41, R42, R43, R44, R45, R46, R47, R48, R49: symbol CellsBoard:R -> Device:R
Connections:
- net CB0: no longer RN1.1 (R1.1), RN1.2 (R2.1), RN1.7 (R2.2), RN1.8 (R1.2)
- no-connect marks 0 -> 4
Other:
- note removed: "DUAL RESISTOR = POPULATE THE RESISTOR FROM R1 TO R18 + FROM R32 TO R49"
- note removed: "SINGLE RESISTOR = POPULATE ONLY THE RESISTOR FROM R1 TO R18"
