File: cellboard/CellsBoard.kicad_pcb (KiCad board)
At the start: 2 copper layers, 445.5 x 71.5 mm, 268 parts, among them CN1 10nF_array, CN2 10nF_array, CN3 10nF_array, CN4 10nF_array, CN5 10nF_array, J1 Conn_02x08, J10 BUS, J19 CONN_1X02, J2 Conn_02x08, J20 CONN_1X02, J3 Conn_02x08, J4 Conn_02x08, J5 Conn_02x08, J7 CONN_1x08, J8 CONN_1X02, J9 BUS, Q1 BSS308PE, Q10 BSS308PE, Q11 BSS308PE, Q12 BSS308PE, Q13 BSS308PE, Q14 BSS308PE, Q15 BSS308PE, Q16 BSS308PE, Q17 BSS308PE, Q18 BSS308PE, Q19 TSM3401CX RFG, Q2 BSS308PE, Q20 TSM3401CX RFG, Q21 TSM3401CX RFG, Q22 TSM3401CX RFG, Q23 TSM3401CX RFG, Q3 BSS308PE, Q4 BSS308PE, Q5 BSS308PE, Q6 BSS308PE, Q7 BSS308PE, Q8 BSS308PE, Q9 BSS308PE, SW1 RESET, T40 TestPoint, U1 LTC6813-1, U10 M95256-W, U11 MAX14878AWA+, U12 ADC128D818, U13 ADC128D818, U14 ADC128D818, U15 CellBoardConnection, U2 MCP1812, U3 HM2103, U4 HM2103, U5 STM32G474CxU, U6 ADC128D818, U7 ADC128D818, U8 LT8630, U9 LTC3639

Commit message: v2.1.2.5 as printed
Commit on behalf of fran-retfie.
Parts:
- removed D1: BAS16J, Diode_SMD:D_SOD-323
- removed J19, J20: CONN_1X02, CellsBoard:Molex_Micro-Fit_3.0_43650-0215_1x02_P3.00mm_Vertical
- removed JP10, JP11, JP12, JP13, JP14, JP15, JP16, JP17, JP18, JP6, JP7, JP8, JP9: Jumper_NC_Small, CellsBoard:JUMPER_NC
- removed JP19: GND_connection, CellsBoard:I2C_JUMPER_CONNECTION
- removed JP21: SolderJumper_3_Open, CellsBoard:PinHeader_1x03_P2.54mm_Vertical
- removed JP25: SPI, CellsBoard:Jumper_adafruit
- removed L2: 560uH, CellsBoard:Inductor_Bourns_SRR4028
- removed Q19, Q20, Q21, Q22, Q23: TSM3401CX RFG, CellsBoard:SOT-23
- removed R10, R11, R12, R13, R14, R15, R16, R17, R18, R9: Rdsc, Resistor_SMD:R_2512_6332Metric
- removed R20: 100, Resistor_SMD:R_0805_2012Metric
- removed R21: 25K5, Resistor_SMD:R_0603_1608Metric
- removed R22, R50: 1M, Resistor_SMD:R_0603_1608Metric
- removed R23: 191k, Resistor_SMD:R_0603_1608Metric
- removed R28, R29, R30, R31: 150, Resistor_SMD:R_0603_1608Metric
- removed T40: TestPoint, CellsBoard:Test_point
- added C84: 10n, Capacitor_SMD:C_0805_2012Metric, F.Cu at (96.9, 130.3)
- added C85: 100nF, Capacitor_SMD:C_0603_1608Metric, F.Cu at (179.4, 137.5)
- added C86: 100nF, Capacitor_SMD:C_0603_1608Metric, F.Cu at (163.6, 144.3)
- added C87: 100nF, Capacitor_SMD:C_0603_1608Metric, F.Cu at (156.1, 139.7)
- added F21: Fuse, CellsBoard:Fuse_0805, F.Cu at (350.8, 157.4)
- added F22: Fuse, CellsBoard:Fuse_0805, F.Cu at (276.8, 157.7)
- added F23: Fuse, CellsBoard:Fuse_0805, F.Cu at (201.5, 157.2)
- added F24: Fuse, CellsBoard:Fuse_0805, F.Cu at (127.4, 158.0)
- added F25: Fuse, CellsBoard:Fuse_0805, F.Cu at (508.2, 152.6)
- added J11: Conn_02x06_Top_Bottom, Connector_Molex:Molex_Nano-Fit_105310-xx12_2x06_P2.50mm_Vertical, F.Cu at (312.8, 165.7)
- added J12: Conn_02x06_Top_Bottom, Connector_Molex:Molex_Nano-Fit_105310-xx12_2x06_P2.50mm_Vertical, F.Cu at (387.5, 165.6)
- added J13: Conn_02x06_Top_Bottom, Connector_Molex:Molex_Nano-Fit_105310-xx12_2x06_P2.50mm_Vertical, F.Cu at (164.5, 165.6)
- added J14: Conn_02x06_Top_Bottom, Connector_Molex:Molex_Nano-Fit_105310-xx12_2x06_P2.50mm_Vertical, F.Cu at (90.0, 165.6)
- added J15: Conn_02x06_Top_Bottom, Connector_Molex:Molex_Nano-Fit_105310-xx12_2x06_P2.50mm_Vertical, F.Cu at (239.9, 165.6)
- added J16: Conn_02x06_Top_Bottom, Connector_Molex:Molex_Nano-Fit_105310-xx12_2x06_P2.50mm_Vertical, F.Cu at (461.0, 165.6)
- added J6: Conn_02x02_Odd_Even, Connector_Molex:Molex_Micro-Fit_3.0_43045-0412_2x02_P3.00mm_Vertical, F.Cu at (126.5, 166.2)
- added NT0: Net-Tie_2, NetTie:NetTie-2_SMD_Pad0.5mm, F.Cu at (115.2, 155.8)
- added NT1: Net-Tie_2, NetTie:NetTie-2_SMD_Pad0.5mm, F.Cu at (116.5, 153.2)
- added NT10: Net-Tie_2, NetTie:NetTie-2_SMD_Pad0.5mm, F.Cu at (329.7, 166.4)
- added NT11: Net-Tie_2, NetTie:NetTie-2_SMD_Pad0.5mm, F.Cu at (359.0, 159.6)
- added NT12: Net-Tie_2, NetTie:NetTie-2_SMD_Pad0.5mm, F.Cu at (350.6, 154.6)
- added NT13: Net-Tie_2, NetTie:NetTie-2_SMD_Pad0.5mm, F.Cu at (404.1, 161.6)
- added NT14: Net-Tie_2, NetTie:NetTie-2_SMD_Pad0.5mm, F.Cu at (406.7, 153.5)
- added NT15: Net-Tie_2, NetTie:NetTie-2_SMD_Pad0.5mm, F.Cu at (423.5, 153.7)
- added NT16: Net-Tie_2, NetTie:NetTie-2_SMD_Pad0.5mm, F.Cu at (482.2, 162.4)
- added NT17: Net-Tie_2, NetTie:NetTie-2_SMD_Pad0.5mm, F.Cu at (507.6, 159.8)
- added NT18: Net-Tie_2, NetTie:NetTie-2_SMD_Pad0.5mm, F.Cu at (502.3, 150.5)
- added NT19: Net-Tie_2, NetTie:NetTie-2_SMD_Pad0.5mm, F.Cu at (117.5, 160.4)
- added NT2: Net-Tie_2, NetTie:NetTie-2_SMD_Pad0.5mm, F.Cu at (134.2, 155.2)
- added NT20: Net-Tie_2, NetTie:NetTie-2_SMD_Pad2.0mm, F.Cu at (134.3, 133.6)
- added NT3: Net-Tie_2, NetTie:NetTie-2_SMD_Pad0.5mm, F.Cu at (201.1, 151.0)
- added NT4: Net-Tie_2, NetTie:NetTie-2_SMD_Pad0.5mm, F.Cu at (185.1, 159.0)
- added NT5: Net-Tie_2, NetTie:NetTie-2_SMD_Pad0.5mm, F.Cu at (211.4, 159.4)
- added NT6: Net-Tie_2, NetTie:NetTie-2_SMD_Pad0.5mm, F.Cu at (210.2, 155.6)
- added NT7: Net-Tie_2, NetTie:NetTie-2_SMD_Pad0.5mm, F.Cu at (265.6, 150.0)
- added NT8: Net-Tie_2, NetTie:NetTie-2_SMD_Pad0.5mm, F.Cu at (286.5, 161.7)
- added NT9: Net-Tie_2, NetTie:NetTie-2_SMD_Pad0.5mm, F.Cu at (276.4, 150.4)
- added TP10: 5V_ISO, TestPoint:TestPoint_Pad_D1.0mm, F.Cu at (158.3, 114.2)
- added TP11: GND_ISO, TestPoint:TestPoint_Pad_D1.0mm, F.Cu at (163.8, 114.2)
- added TP12: VCC, TestPoint:TestPoint_Pad_D1.0mm, F.Cu at (505.4, 140.8)
- added TP3: TestPoint, CellsBoard:TestPoint_GNDedge_toponly, F.Cu at (145.8, 175.7)
- added TP4: TestPoint, CellsBoard:TestPoint_GNDedge_toponly, F.Cu at (361.8, 175.7)
- added TP6: VRef2, TestPoint:TestPoint_Pad_D1.0mm, F.Cu at (246.3, 143.9)
- added TP7: TestPoint, CellsBoard:TestPoint_GNDedge_toponly, F.Cu at (127.6, 106.3)
- added TP8: V+, TestPoint:TestPoint_Pad_D1.0mm, F.Cu at (265.2, 143.4)
- added TP9: +5V, TestPoint:TestPoint_Pad_D1.0mm, F.Cu at (126.0, 137.0)
- added U16: MCP1811AT-033LT, Package_TO_SOT_SMD:SOT-23-5_HandSoldering, F.Cu at (387.4, 147.6)
- added U17: MCP1811AT-033LT, Package_TO_SOT_SMD:SOT-23-5_HandSoldering, F.Cu at (172.0, 150.6)
- added U18: MCP1811AT-033LT, Package_TO_SOT_SMD:SOT-23-5_HandSoldering, F.Cu at (91.2, 147.7)
- added U19: MCP1811AT-033LT, Package_TO_SOT_SMD:SOT-23-5_HandSoldering, F.Cu at (258.0, 163.6)
- added U20: MCP1811AT-033LT, Package_TO_SOT_SMD:SOT-23-5_HandSoldering, F.Cu at (461.9, 148.1)
- added U21: DSC61XX, CellsBoard:4-Lead_CDFN_2.5x2.0mm, F.Cu at (170.7, 139.8)
- C10, C27, C29, C43, C55: value 100nF -> 1uF
- C19: value 100nF -> 22n; footprint Capacitor_SMD:C_0603_1608Metric -> Capacitor_SMD:C_0603_1608Metric_Pad1.08x0.95mm_HandSolder
- C23: value 4.7uF -> 10n; footprint Capacitor_SMD:C_1210_3225Metric -> Capacitor_SMD:C_0805_2012Metric_Pad1.18x1.45mm_HandSolder
- C24: value 22uF -> 1u; footprint Capacitor_SMD:C_1210_3225Metric -> Capacitor_SMD:C_0805_2012Metric_Pad1.18x1.45mm_HandSolder
- C25: value 100nF -> 47u; footprint Capacitor_SMD:C_0603_1608Metric -> Capacitor_SMD:C_1210_3225Metric_Pad1.33x2.70mm_HandSolder
- C26, C28: value 1uF -> 100nF
- C37: value 4.7uF -> 100nF; footprint Capacitor_SMD:C_1210_3225Metric -> Capacitor_SMD:C_0603_1608Metric
- C38: value 100pF -> 100nF
- C39: value 2.2uF -> 100nF
- C40: value 10pF -> 100nF
- C41: value 22uF -> 100nF; footprint Capacitor_SMD:C_1210_3225Metric -> Capacitor_SMD:C_0603_1608Metric
- C42: value 100nF_HV -> 100nF; footprint Capacitor_SMD:C_1206_3216Metric -> Capacitor_SMD:C_0603_1608Metric
- C66: value 100nF -> 10n; footprint Capacitor_SMD:C_0603_1608Metric -> Capacitor_SMD:C_0805_2012Metric_Pad1.18x1.45mm_HandSolder
- C67: value 100nF -> 3n; footprint Capacitor_SMD:C_0603_1608Metric -> Capacitor_SMD:C_0805_2012Metric_Pad1.18x1.45mm_HandSolder
- C78: value 100nF -> 1u_HV; footprint Capacitor_SMD:C_0603_1608Metric -> Capacitor_SMD:C_2220_5650Metric_Pad1.97x5.40mm_HandSolder
- C79: value 100nF -> 100n; footprint Capacitor_SMD:C_0603_1608Metric -> Capacitor_SMD:C_0805_2012Metric
- C8, C9: value 10nF -> 1u_HV; footprint Capacitor_SMD:C_0603_1608Metric -> Capacitor_SMD:C_2220_5650Metric_Pad1.97x5.40mm_HandSolder
- J1, J2, J3, J4, J5: value Conn_02x08 -> Conn_02x02_Odd_Even; footprint CellsBoard:Molex_Micro-Fit_3.0_43045-1612_2x08_P3.00mm_Vertical -> Connector_Molex:Molex_Micro-Fit_3.0_43045-0412_2x02_P3.00mm_Vertical
- J7: value CONN_1x08 -> Conn_02x05_Top_Bottom; footprint Connector_PinHeader_1.27mm:PinHeader_1x08_P1.27mm_Vertical -> Connector_Molex:Molex_Nano-Fit_105310-xx10_2x05_P2.50mm_Vertical
- J8: value CONN_1X02 -> Conn_02x02_Counter_Clockwise; footprint CellsBoard:Molex_Micro-Fit_3.0_43650-0215_1x02_P3.00mm_Vertical -> Connector_Molex:Molex_Micro-Fit_3.0_43045-0412_2x02_P3.00mm_Vertical
- JP1, JP2, JP3, JP4: value Jumper_NC_Small -> SolderJumper_3_Open; footprint CellsBoard:JUMPER_NC -> Jumper:SolderJumper-3_P1.3mm_Open_RoundedPad1.0x1.5mm
- JP5: value Jumper_NC_Small -> SolderJumper_2_Open; footprint CellsBoard:JUMPER_NC -> Jumper:SolderJumper-2_P1.3mm_Open_RoundedPad1.0x1.5mm
- L1: value 22uH -> 56u; footprint CellsBoard:SLF10145_Type_BigPad -> CellsBoard:sdr1307
- Q1, Q10, Q11, Q12, Q13, Q14, Q2, Q3, Q4, Q5, Q6, Q7, Q8, Q9: value BSS308PE -> TSM3401CX RFG
- R1: value Rdsc -> 100; footprint Resistor_SMD:R_2512_6332Metric -> Resistor_SMD:R_0603_1608Metric
- R2: value Rdsc -> 1.24k; footprint Resistor_SMD:R_2512_6332Metric -> Resistor_SMD:R_0805_2012Metric_Pad1.20x1.40mm_HandSolder
- R24: value 1k4 -> 1k
- R25: value 604 -> 1k
- R3: value Rdsc -> 100k; footprint Resistor_SMD:R_2512_6332Metric -> Resistor_SMD:R_0805_2012Metric_Pad1.20x1.40mm_HandSolder
- R32, R33, R34, R35, R36, R37, R38, R39, R40, R41, R43, R44, R45, R46, R47, R48, R49: moved to F.Cu
- R4: value Rdsc -> 2k; footprint Resistor_SMD:R_2512_6332Metric -> Resistor_SMD:R_0805_2012Metric_Pad1.20x1.40mm_HandSolder
- R5: value Rdsc -> 215k; footprint Resistor_SMD:R_2512_6332Metric -> Resistor_SMD:R_0805_2012Metric_Pad1.20x1.40mm_HandSolder
- R6: value Rdsc -> 3k; footprint Resistor_SMD:R_2512_6332Metric -> Resistor_SMD:R_0603_1608Metric_Pad0.98x0.95mm_HandSolder
- R7: value Rdsc -> 2k; footprint Resistor_SMD:R_2512_6332Metric -> Resistor_SMD:R_0603_1608Metric_Pad0.98x0.95mm_HandSolder
- R8: value Rdsc -> 255k; footprint Resistor_SMD:R_2512_6332Metric -> Resistor_SMD:R_0805_2012Metric_Pad1.20x1.40mm_HandSolder
- RN11, RN14, RN17, RN18, RN19, RN20, RN21, RN22, RN23, RN24: value 3K3 -> x; footprint Resistor_SMD:R_Array_Convex_4x1206 -> Resistor_SMD:R_Array_Convex_4x0603
- RN15, RN16: value 0 ohm -> x; footprint Resistor_SMD:R_Array_Convex_2x0603 -> Resistor_SMD:R_Array_Convex_4x0603
- TP1, TP2: footprint CellsBoard:Test_point -> CellsBoard:TestPoint_GNDedge_toponly
- TP5: value TestPoint -> VRef1; footprint CellsBoard:Test_point -> TestPoint:TestPoint_Pad_D1.0mm
- U11: footprint Package_SO:SOIC-8_7.5x5.85mm_P1.27mm -> Package_SO:SOIC-8_5.23x5.23mm_P1.27mm
- U15: value CellBoardConnection -> MCP1811AT-033LT; footprint CellsBoard:CELL_SPACE_FINAL -> Package_TO_SOT_SMD:SOT-23-5_HandSoldering
- U2: footprint Package_TO_SOT_SMD:SOT-323_SC-70 -> Package_TO_SOT_SMD:SOT-23_Handsoldering
- U3: value HM2103 -> CPC1125N; footprint CellsBoard:HM2103 -> Package_SO:SOP-4_3.8x4.1mm_P2.54mm
- U4: value HM2103 -> LM5161PWP; footprint CellsBoard:HM2103 -> Package_SO:HTSSOP-14-1EP_4.4x5mm_P0.65mm_EP3.4x5mm_Mask3x3.1mm
- U5: value STM32G474CxU -> STM32L432KBUx; footprint Package_QFP:LQFP-48_7x7mm_P0.5mm -> Package_DFN_QFN:QFN-32-1EP_5x5mm_P0.5mm_EP3.45x3.45mm
- U8: value LT8630 -> MAQ5281; footprint CellsBoard:LT8631 -> Package_SO:MSOP-8-1EP_3x3mm_P0.65mm_EP1.68x1.88mm
- U9: value LTC3639 -> ADC128D818; footprint CellsBoard:MSOP-12-16-1EP_3x4mm_P0.5mm_EP1.65x2.85mm_ThermalVias -> CellsBoard:TSSOP-16_4.4x5mm_P0.65mm
- moved J8 403.9 mm to (100.6, 113.5), turned to 180 degrees
- moved C24 382.9 mm to (116.6, 112.5), turned to 0 degrees
- moved C23 377.3 mm to (116.6, 115.6), turned to 90 degrees
- moved C67 353.7 mm to (107.6, 126.8), turned to 270 degrees
- moved C66 347.1 mm to (116.6, 110.1), turned to 180 degrees
- moved U8 315.0 mm to (101.3, 128.5), turned to 270 degrees
- moved L1 312.7 mm to (116.9, 125.0)
- moved C19 275.0 mm to (127.0, 109.8), turned to 0 degrees
- moved C25 270.4 mm to (128.3, 129.6)
- moved C80 243.3 mm to (94.4, 148.7), turned to 270 degrees
- moved RN23 242.5 mm to (95.1, 152.1), turned to 270 degrees
- moved C73 241.1 mm to (100.5, 158.0)
- moved C72 240.8 mm to (102.1, 158.0), turned to 270 degrees
- moved C74 240.5 mm to (97.0, 158.0), turned to 270 degrees
- moved C81 239.2 mm to (96.4, 148.7), turned to 270 degrees
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Connections:
- net /BATTERY MANAGER/Cell0 renamed /BATTERY MANAGER/C0
- net /BATTERY MANAGER/Cell1 renamed /BATTERY MANAGER/C1
- net /BATTERY MANAGER/Cell10 renamed /BATTERY MANAGER/C10
- net /BATTERY MANAGER/Cell11 renamed /BATTERY MANAGER/C11
- net /BATTERY MANAGER/Cell12 renamed /BATTERY MANAGER/C12
- net /BATTERY MANAGER/Cell13 renamed /BATTERY MANAGER/C13
- net /BATTERY MANAGER/Cell14 renamed /BATTERY MANAGER/C14
- net /BATTERY MANAGER/Cell15 renamed /BATTERY MANAGER/C15
- net /BATTERY MANAGER/Cell16 renamed /BATTERY MANAGER/C16
- net /BATTERY MANAGER/Cell17 renamed /BATTERY MANAGER/C17
- net /BATTERY MANAGER/Cell18 renamed /BATTERY MANAGER/C18
- net /BATTERY MANAGER/Cell2 renamed /BATTERY MANAGER/C2
- net /BATTERY MANAGER/Cell3 renamed /BATTERY MANAGER/C3
- net /BATTERY MANAGER/Cell4 renamed /BATTERY MANAGER/C4
- net /BATTERY MANAGER/Cell5 renamed /BATTERY MANAGER/C5
- net /BATTERY MANAGER/Cell6 renamed /BATTERY MANAGER/C6
- net /BATTERY MANAGER/Cell7 renamed /BATTERY MANAGER/C7
- net /BATTERY MANAGER/Cell8 renamed /BATTERY MANAGER/C8
- net /BATTERY MANAGER/Cell9 renamed /BATTERY MANAGER/C9
- net /BATTERY MANAGER/Temperature/~W~ renamed /STM/~W~
- C1 pad 1: +3V3 -> GND
- C1 pad 2: GND -> +3V3
- C13 pad 1: /BATTERY MANAGER/Temperature/RESET -> /STM/RESET
- C19 pad 1: Net-(C19-Pad1) -> /DCDC_80Vto5V/GND_SUPPLY
- C19 pad 2: GND -> /DCDC_80Vto5V/SS-D
- C20 pad 1: +3V3 -> GND
- C20 pad 2: GND -> +3V3
- C23 pad 1: /BATTERY MANAGER/CB18 -> /DCDC_80Vto5V/SW-D
- C23 pad 2: GND -> Net-(C23-Pad2)
- C24 pad 1: Net-(C24-Pad1) -> /DCDC_80Vto5V/GND_SUPPLY
- C24 pad 2: GND -> /DCDC_80Vto5V/VCC-D
- C25 pad 1: Net-(C25-Pad1) -> /DCDC_80Vto5V/GND_SUPPLY
- C25 pad 2: GND -> +5V
- C26 pad 2: Net-(C26-Pad2) -> /STM/temperatureADC_3/3V3_SENS
- C27 pad 2: Net-(C26-Pad2) -> /STM/temperatureADC_3/3V3_SENS
- C28 pad 2: +3V3 -> +5V
- C29 pad 2: +3V3 -> +5V
- C37 pad 1: /BATTERY MANAGER/DCDC_80Vto5V/VIN -> Net-(C37-Pad1)
- C37 pad 2: /BATTERY MANAGER/0V -> GND
- C38 pad 1: /BATTERY MANAGER/DCDC_80Vto5V/TR -> Net-(C38-Pad1)
- C38 pad 2: /BATTERY MANAGER/0V -> GND
- C39 pad 1: /BATTERY MANAGER/0V -> Net-(C39-Pad1)
- C39 pad 2: /BATTERY MANAGER/DCDC_80Vto5V/Int_VCC -> GND
- C40 pad 1: /BATTERY MANAGER/DCDC_80Vto5V/5V -> Net-(C40-Pad1)
- C40 pad 2: /BATTERY MANAGER/DCDC_80Vto5V/FB -> GND
- C41 pad 1: /BATTERY MANAGER/DCDC_80Vto5V/5V -> Net-(C41-Pad1)
- C41 pad 2: /BATTERY MANAGER/0V -> GND
- C42 pad 1: /BATTERY MANAGER/DCDC_80Vto5V/SW -> GND
- C42 pad 2: /BATTERY MANAGER/DCDC_80Vto5V/BST -> /STM/temperatureADC_2/3V3_SENS
- C43 pad 1: Net-(C43-Pad1) -> GND
- C43 pad 2: GND -> /STM/temperatureADC_2/3V3_SENS
- C44 pad 2: Net-(C44-Pad2) -> /STM/temperatureADC_4/3V3_SENS
- C45 pad 2: Net-(C44-Pad2) -> /STM/temperatureADC_4/3V3_SENS
- C46 pad 2: +3V3 -> +5V
- C47 pad 2: +3V3 -> +5V
- C54 pad 1: Net-(C54-Pad1) -> GND
- C54 pad 2: GND -> +5V
- C55 pad 1: Net-(C55-Pad1) -> GND
- C55 pad 2: GND -> +5V
- C56 pad 2: Net-(C56-Pad2) -> /STM/temperatureADC_1/3V3_SENS
- C57 pad 2: Net-(C56-Pad2) -> /STM/temperatureADC_1/3V3_SENS
- C58 pad 2: +3V3 -> +5V
- C59 pad 2: +3V3 -> +5V
- C66 pad 1: Net-(C66-Pad1) -> /DCDC_80Vto5V/FB-D
- C66 pad 2: GND -> Net-(C66-Pad2)
- C67 pad 1: Net-(C67-Pad1) -> Net-(C66-Pad2)
- C67 pad 2: GND -> +5V
- C68 pad 2: Net-(C68-Pad2) -> /STM/temperatureADC_5/3V3_SENS
- C69 pad 2: Net-(C68-Pad2) -> /STM/temperatureADC_5/3V3_SENS
- C70 pad 2: +3V3 -> +5V
- C71 pad 2: +3V3 -> +5V
- C78 pad 1: Net-(C78-Pad1) -> /DCDC_80Vto5V/GND_SUPPLY
- C78 pad 2: GND -> /DCDC_80Vto5V/120V_linreg
- C79 pad 2: GND -> /DCDC_80Vto5V/GND_SUPPLY
- C8 pad 1: GND -> /DCDC_80Vto5V/GND_SUPPLY
- C8 pad 2: Net-(C8-Pad2) -> VCC
- C80 pad 2: Net-(C80-Pad2) -> /STM/temperatureADC_0/3V3_SENS
- C81 pad 2: Net-(C80-Pad2) -> /STM/temperatureADC_0/3V3_SENS
- C82 pad 2: +3V3 -> +5V
- C83 pad 2: +3V3 -> +5V
- C9 pad 1: GND -> /DCDC_80Vto5V/GND_SUPPLY
- C9 pad 2: Net-(C9-Pad2) -> VCC
- F1 pad 2: GND -> /CB0
- F10 pad 1: /CB9N -> /CB9N-2
- F13 pad 1: /CB12N -> /CB12N-1
- F16 pad 1: /CB15N -> /CB15N-1
- F20 pad 1: +5V -> /CB15N-2
- F20 pad 2: /BATTERY MANAGER/DCDC_80Vto5V/5V -> /CB15
- F4 pad 1: /CB3N -> /CB3N-1
- F7 pad 1: /CB6N -> /CB6N-1
- J1 pad 1: GND -> /CB17N
- J1 pad 2: GND -> /CB16N
- J1 pad 3: GND -> /CB18N
- J1 pad 4: GND -> /CB15N-1
- J10 pad 1: /BATTERY MANAGER/Temperature/5V_ISO -> /STM/CANL_ISO
- J10 pad 2: /BATTERY MANAGER/Temperature/GND_ISO -> /STM/CANH_ISO
- J10 pad 3: /BATTERY MANAGER/Temperature/CANH_ISO -> /DCDC_80Vto5V/GND_ISO
- J10 pad 4: /BATTERY MANAGER/Temperature/CANL_ISO -> /DCDC_80Vto5V/5V_ISO
- J2 pad 1: GND -> /CB14N
- J2 pad 2: GND -> /CB13N
- J2 pad 3: GND -> /CB15N-2
- J2 pad 4: GND -> /CB12N-1
- J3 pad 1: GND -> /CB11N
- J3 pad 2: GND -> /CB10N
- J3 pad 3: GND -> /CB12N-2
- J3 pad 4: GND -> /CB9N-2
- J4 pad 1: GND -> /CB8N
- J4 pad 2: GND -> /CB7N
- J4 pad 3: GND -> /CB9N-1
- J4 pad 4: GND -> /CB6N-1
- J5 pad 1: GND -> /CB5N
- J5 pad 2: GND -> /CB4N
- J5 pad 3: GND -> /CB6N-2
- J5 pad 4: GND -> /CB3N-1
- J7 pad 2: +3V3 -> /STM/SWCLK
- J7 pad 3: /BATTERY MANAGER/Temperature/SWO -> /STM/SWDIO
- J7 pad 4: /BATTERY MANAGER/Temperature/SWCLK -> +3V3
- J7 pad 5: /BATTERY MANAGER/Temperature/SWDIO -> /STM/TX
- J7 pad 6: /BATTERY MANAGER/Temperature/RESET -> GND
- J7 pad 7: /BATTERY MANAGER/Temperature/TX -> /STM/RESET
- J7 pad 8: /BATTERY MANAGER/Temperature/RX -> /STM/SWO
- J8 pad 1: Net-(C24-Pad1) -> Net-(C84-Pad1)
- J8 pad 2: GND -> /DCDC_80Vto5V/GND_SUPPLY
- J9 pad 1: /BATTERY MANAGER/Temperature/5V_ISO -> /STM/CANL_ISO
- J9 pad 2: /BATTERY MANAGER/Temperature/GND_ISO -> /STM/CANH_ISO
- J9 pad 3: /BATTERY MANAGER/Temperature/CANH_ISO -> /DCDC_80Vto5V/GND_ISO
- J9 pad 4: /BATTERY MANAGER/Temperature/CANL_ISO -> /DCDC_80Vto5V/5V_ISO
- JP1 pad 1: /CB1 -> GND
- JP1 pad 2: /BATTERY MANAGER/CB1 -> /STM/ADD_0
- JP2 pad 1: /CB2 -> /STM/SCK_EEPROM
- JP2 pad 2: /BATTERY MANAGER/CB2 -> Net-(JP2-Pad2)
- JP3 pad 1: /CB3 -> GND
- JP3 pad 2: /BATTERY MANAGER/CB3 -> /STM/ADD_1
- JP4 pad 1: /CB4 -> GND
- JP4 pad 2: /BATTERY MANAGER/CB4 -> /STM/ADD_2
- JP5 pad 1: /CB5 -> Net-(JP5-Pad1)
- JP5 pad 2: /BATTERY MANAGER/CB5 -> /DCDC_80Vto5V/VCC-D
- L1 pad 1: /BATTERY MANAGER/DCDC_80Vto5V/SW -> /DCDC_80Vto5V/SW-D
- L1 pad 2: /BATTERY MANAGER/DCDC_80Vto5V/IND -> +5V
- R1 pad 1: GND -> Net-(R1-Pad1)
- R1 pad 2: /MOS_Balancer_Passive_metod/DIS_1 -> Net-(R1-Pad2)
- R2 pad 1: /CB1 -> Net-(R2-Pad1)
- R2 pad 2: /MOS_Balancer_Passive_metod/DIS_2 -> /DCDC_80Vto5V/GND_ISO
- R27 pad 2: /BATTERY MANAGER/CB18 -> VCC
- R3 pad 1: /CB2 -> /DCDC_80Vto5V/EN-D
- R3 pad 2: /MOS_Balancer_Passive_metod/DIS_3 -> /DCDC_80Vto5V/EN-DCDC1
- R32 pad 1: GND -> /CB0
- R4 pad 1: /CB3 -> /DCDC_80Vto5V/GND_SUPPLY
- R4 pad 2: /MOS_Balancer_Passive_metod/DIS_4 -> /DCDC_80Vto5V/EN-D
- R5 pad 1: /CB4 -> VCC
- R5 pad 2: /MOS_Balancer_Passive_metod/DIS_5 -> Net-(R5-Pad2)
- R52 pad 1: /BATTERY MANAGER/Temperature/CANH_ISO -> /STM/CANH_ISO
- R52 pad 2: /BATTERY MANAGER/Temperature/CANL_ISO -> /STM/CANL_ISO
- R53 pad 1: /BATTERY MANAGER/MISO -> +3V3
- R53 pad 2: +3V3 -> /BATTERY MANAGER/MISO
- R54 pad 1: /BATTERY MANAGER/Temperature/ADC_nINT -> /STM/ADC_nINT
- R6 pad 1: /CB5 -> +5V
- R6 pad 2: /MOS_Balancer_Passive_metod/DIS_6 -> /DCDC_80Vto5V/FB-D
- R7 pad 1: /CB6 -> /DCDC_80Vto5V/FB-D
- R7 pad 2: /MOS_Balancer_Passive_metod/DIS_7 -> /DCDC_80Vto5V/GND_SUPPLY
- R8 pad 1: /CB7 -> Net-(C66-Pad2)
- R8 pad 2: /MOS_Balancer_Passive_metod/DIS_8 -> /DCDC_80Vto5V/SW-D
- RN1 pad 1: GND -> Net-(RN1-Pad1)
- RN1 pad 2: GND -> Net-(RN1-Pad2)
- RN1 pad 7: GND -> Net-(RN1-Pad7)
- RN1 pad 8: GND -> Net-(RN1-Pad8)
- RN10 pad 3: GND -> /BATTERY MANAGER/CB0
- RN11 pad 1: Net-(C26-Pad2) -> /STM/temperatureADC_3/3V3_SENS
- RN11 pad 2: Net-(C26-Pad2) -> /STM/temperatureADC_3/3V3_SENS
- RN11 pad 3: Net-(C26-Pad2) -> /STM/temperatureADC_3/3V3_SENS
- RN11 pad 4: Net-(C26-Pad2) -> /STM/temperatureADC_3/3V3_SENS
- RN11 pad 5: Net-(C11-Pad1) -> Net-(C16-Pad1)
- RN11 pad 6: Net-(C14-Pad1) -> Net-(C15-Pad1)
- RN11 pad 7: Net-(C15-Pad1) -> Net-(C14-Pad1)
- RN11 pad 8: Net-(C16-Pad1) -> Net-(C11-Pad1)
- RN12 pad 3: /BATTERY MANAGER/SCL -> /STM/SDA
- RN12 pad 4: /BATTERY MANAGER/SDA -> /STM/SCL
- RN13 pad 5: /BATTERY MANAGER/Temperature/CS_EEPROM -> /STM/CS_EEPROM
- RN13 pad 6: /BATTERY MANAGER/Temperature/MISO_EEPROM -> /STM/MISO_EEPROM
- RN13 pad 7: /BATTERY MANAGER/Temperature/~HOLD~ -> /STM/~HOLD~
- RN13 pad 8: /BATTERY MANAGER/Temperature/SCK_EEPROM -> /STM/SCK_EEPROM
- RN14 pad 1: Net-(C26-Pad2) -> /STM/temperatureADC_3/3V3_SENS
- RN14 pad 2: Net-(C26-Pad2) -> /STM/temperatureADC_3/3V3_SENS
- RN14 pad 3: Net-(C26-Pad2) -> /STM/temperatureADC_3/3V3_SENS
- RN14 pad 4: Net-(C26-Pad2) -> GND
- RN14 pad 5: Net-(C17-Pad1) -> /STM/temperatureADC_3/A1
- RN14 pad 6: Net-(C18-Pad1) -> /STM/temperatureADC_3/A1
- RN14 pad 7: Net-(C19-Pad1) -> Net-(C18-Pad1)
- RN14 pad 8: Net-(C25-Pad1) -> Net-(C17-Pad1)
- RN15 pad 1: Net-(RN15-Pad1) -> /STM/temperatureADC_2/3V3_SENS
- RN15 pad 2: Net-(RN15-Pad2) -> /STM/temperatureADC_2/3V3_SENS
- RN15 pad 3: /BATTERY MANAGER/CLK -> /STM/temperatureADC_2/3V3_SENS
- RN15 pad 4: /BATTERY MANAGER/~CS~ -> /STM/temperatureADC_2/3V3_SENS
- RN16 pad 1: Net-(RN15-Pad2) -> /STM/temperatureADC_2/3V3_SENS
- RN16 pad 2: Net-(RN15-Pad1) -> /STM/temperatureADC_2/3V3_SENS
- RN16 pad 3: /BATTERY MANAGER/IMA -> /STM/temperatureADC_2/3V3_SENS
- RN16 pad 4: /BATTERY MANAGER/IPA -> GND
- RN17 pad 1: Net-(C44-Pad2) -> /STM/temperatureADC_4/3V3_SENS
- RN17 pad 2: Net-(C44-Pad2) -> /STM/temperatureADC_4/3V3_SENS
- RN17 pad 3: Net-(C44-Pad2) -> /STM/temperatureADC_4/3V3_SENS
- RN17 pad 4: Net-(C44-Pad2) -> /STM/temperatureADC_4/3V3_SENS
- RN17 pad 5: Net-(C30-Pad1) -> Net-(C33-Pad1)
- RN17 pad 6: Net-(C31-Pad1) -> Net-(C32-Pad1)
- RN17 pad 7: Net-(C32-Pad1) -> Net-(C31-Pad1)
- RN17 pad 8: Net-(C33-Pad1) -> Net-(C30-Pad1)
- RN18 pad 1: Net-(C44-Pad2) -> /STM/temperatureADC_4/3V3_SENS
- RN18 pad 2: Net-(C44-Pad2) -> /STM/temperatureADC_4/3V3_SENS
- RN18 pad 3: Net-(C44-Pad2) -> /STM/temperatureADC_4/3V3_SENS
- RN18 pad 4: Net-(C44-Pad2) -> GND
- RN18 pad 5: Net-(C34-Pad1) -> /STM/temperatureADC_4/A0
- RN18 pad 6: Net-(C35-Pad1) -> /STM/temperatureADC_4/A0
- RN18 pad 7: Net-(C36-Pad1) -> Net-(C35-Pad1)
- RN18 pad 8: Net-(C43-Pad1) -> Net-(C34-Pad1)
- RN19 pad 1: Net-(C56-Pad2) -> /STM/temperatureADC_1/3V3_SENS
- RN19 pad 2: Net-(C56-Pad2) -> /STM/temperatureADC_1/3V3_SENS
- RN19 pad 3: Net-(C56-Pad2) -> /STM/temperatureADC_1/3V3_SENS
- RN19 pad 4: Net-(C56-Pad2) -> /STM/temperatureADC_1/3V3_SENS
- RN19 pad 5: Net-(C48-Pad1) -> Net-(C51-Pad1)
- RN19 pad 6: Net-(C49-Pad1) -> Net-(C50-Pad1)
- RN19 pad 7: Net-(C50-Pad1) -> Net-(C49-Pad1)
- RN19 pad 8: Net-(C51-Pad1) -> Net-(C48-Pad1)
- RN20 pad 1: Net-(C56-Pad2) -> /STM/temperatureADC_1/3V3_SENS
- RN20 pad 2: Net-(C56-Pad2) -> /STM/temperatureADC_1/3V3_SENS
- RN20 pad 3: Net-(C56-Pad2) -> /STM/temperatureADC_1/3V3_SENS
- RN20 pad 4: Net-(C56-Pad2) -> GND
- RN20 pad 5: Net-(C52-Pad1) -> /STM/temperatureADC_1/A0
- RN20 pad 6: Net-(C53-Pad1) -> /STM/temperatureADC_1/A0
- RN20 pad 7: Net-(C54-Pad1) -> Net-(C53-Pad1)
- RN20 pad 8: Net-(C55-Pad1) -> Net-(C52-Pad1)
- RN21 pad 1: Net-(C68-Pad2) -> /STM/temperatureADC_5/3V3_SENS
- RN21 pad 2: Net-(C68-Pad2) -> /STM/temperatureADC_5/3V3_SENS
- RN21 pad 3: Net-(C68-Pad2) -> /STM/temperatureADC_5/3V3_SENS
- RN21 pad 4: Net-(C68-Pad2) -> /STM/temperatureADC_5/3V3_SENS
- RN21 pad 5: Net-(C60-Pad1) -> Net-(C63-Pad1)
- RN21 pad 6: Net-(C61-Pad1) -> Net-(C62-Pad1)
- RN21 pad 7: Net-(C62-Pad1) -> Net-(C61-Pad1)
- RN21 pad 8: Net-(C63-Pad1) -> Net-(C60-Pad1)
- RN22 pad 1: Net-(C68-Pad2) -> /STM/temperatureADC_5/3V3_SENS
- RN22 pad 2: Net-(C68-Pad2) -> /STM/temperatureADC_5/3V3_SENS
- RN22 pad 3: Net-(C68-Pad2) -> /STM/temperatureADC_5/3V3_SENS
- RN22 pad 4: Net-(C68-Pad2) -> GND
- RN22 pad 5: Net-(C64-Pad1) -> /STM/temperatureADC_5/A1
- RN22 pad 6: Net-(C65-Pad1) -> /STM/temperatureADC_5/A1
- RN22 pad 7: Net-(C66-Pad1) -> Net-(C65-Pad1)
- RN22 pad 8: Net-(C67-Pad1) -> Net-(C64-Pad1)
- RN23 pad 1: Net-(C80-Pad2) -> /STM/temperatureADC_0/3V3_SENS
- RN23 pad 2: Net-(C80-Pad2) -> /STM/temperatureADC_0/3V3_SENS
- RN23 pad 3: Net-(C80-Pad2) -> /STM/temperatureADC_0/3V3_SENS
- RN23 pad 4: Net-(C80-Pad2) -> /STM/temperatureADC_0/3V3_SENS
- RN23 pad 5: Net-(C72-Pad1) -> Net-(C75-Pad1)
- RN23 pad 6: Net-(C73-Pad1) -> Net-(C74-Pad1)
- RN23 pad 7: Net-(C74-Pad1) -> Net-(C73-Pad1)
- RN23 pad 8: Net-(C75-Pad1) -> Net-(C72-Pad1)
- RN24 pad 1: Net-(C80-Pad2) -> /STM/temperatureADC_0/3V3_SENS
- RN24 pad 2: Net-(C80-Pad2) -> /STM/temperatureADC_0/3V3_SENS
- RN24 pad 3: Net-(C80-Pad2) -> /STM/temperatureADC_0/3V3_SENS
- RN24 pad 4: Net-(C80-Pad2) -> GND
- RN24 pad 5: Net-(C76-Pad1) -> /STM/temperatureADC_0/MID
- RN24 pad 6: Net-(C77-Pad1) -> /STM/temperatureADC_0/MID
- RN24 pad 7: Net-(C78-Pad1) -> Net-(C77-Pad1)
- RN24 pad 8: Net-(C79-Pad1) -> Net-(C76-Pad1)
- SW1 pad 2: /BATTERY MANAGER/Temperature/RESET -> /STM/RESET
- TP1 pad 1: /BATTERY MANAGER/0V -> GND
- TP5 pad 1: +5V -> /BATTERY MANAGER/VRef1
- U1 pad 39: (no net) -> Net-(U1-Pad39)
- U1 pad 40: (no net) -> Net-(U1-Pad40)
- U1 pad 41: (no net) -> Net-(U1-Pad41)
- U1 pad 42: /BATTERY MANAGER/SCL -> Net-(U1-Pad42)
- U1 pad 43: /BATTERY MANAGER/SDA -> Net-(U1-Pad43)
- U1 pad 44: (no net) -> Net-(U1-Pad44)
- U1 pad 45: (no net) -> Net-(U1-Pad45)
- U1 pad 46: (no net) -> Net-(U1-Pad46)
- U1 pad 47: (no net) -> Net-(U1-Pad47)
- U1 pad 49: /BATTERY MANAGER/DRIVE -> Net-(U1-Pad49)
- U1 pad 55: Net-(JP25-Pad2) -> GND
- U1 pad 61: Net-(RN15-Pad1) -> /STM/SPI_CS
- U1 pad 62: Net-(RN15-Pad2) -> /BATTERY MANAGER/CLK
- U1 pad 63: /BATTERY MANAGER/IMB -> Net-(R1-Pad1)
- U1 pad 64: /BATTERY MANAGER/IPB -> Net-(R1-Pad2)
- U10 pad 1: /BATTERY MANAGER/Temperature/CS_EEPROM -> /STM/CS_EEPROM
- U10 pad 2: /BATTERY MANAGER/Temperature/MISO_EEPROM -> /STM/MISO_EEPROM
- U10 pad 5: /BATTERY MANAGER/Temperature/MOSI_EEPROM -> /STM/MOSI_EEPROM
- U10 pad 6: /BATTERY MANAGER/Temperature/SCK_EEPROM -> /STM/SCK_EEPROM
- U10 pad 7: /BATTERY MANAGER/Temperature/~HOLD~ -> /STM/~HOLD~
- U11 pad 1: /BATTERY MANAGER/Temperature/CAN_RX -> /STM/CAN_RX
- U11 pad 2: /BATTERY MANAGER/Temperature/CAN_TX -> /STM/CAN_TX
- U11 pad 5: /BATTERY MANAGER/Temperature/GND_ISO -> /DCDC_80Vto5V/GND_ISO
- U11 pad 6: /BATTERY MANAGER/Temperature/CANL_ISO -> /STM/CANL_ISO
- U11 pad 7: /BATTERY MANAGER/Temperature/CANH_ISO -> /STM/CANH_ISO
- U11 pad 8: /BATTERY MANAGER/Temperature/5V_ISO -> /DCDC_80Vto5V/5V_ISO
- U12 pad 1: Net-(C56-Pad2) -> /STM/temperatureADC_1/3V3_SENS
- U12 pad 10: Net-(C54-Pad1) -> Net-(U12-Pad10)
- U12 pad 2: /BATTERY MANAGER/SDA -> /STM/SDA
- U12 pad 3: /BATTERY MANAGER/SCL -> /STM/SCL
- U12 pad 5: +3V3 -> /STM/temperatureADC_1/3V3_SENS
- U12 pad 6: /BATTERY MANAGER/Temperature/ADC_nINT -> /STM/ADC_nINT
- U12 pad 7: GND -> /STM/temperatureADC_1/A0
- U12 pad 9: Net-(C55-Pad1) -> Net-(U12-Pad9)
- U13 pad 1: Net-(C68-Pad2) -> /STM/temperatureADC_5/3V3_SENS
- U13 pad 10: Net-(C66-Pad1) -> Net-(U13-Pad10)
- U13 pad 2: /BATTERY MANAGER/SDA -> /STM/SDA
- U13 pad 3: /BATTERY MANAGER/SCL -> /STM/SCL
- U13 pad 5: +3V3 -> /STM/temperatureADC_5/3V3_SENS
- U13 pad 6: /BATTERY MANAGER/Temperature/ADC_nINT -> /STM/ADC_nINT
- U13 pad 7: +3V3 -> /STM/temperatureADC_5/3V3_SENS
- U13 pad 8: +3V3 -> /STM/temperatureADC_5/A1
- U13 pad 9: Net-(C67-Pad1) -> Net-(U13-Pad9)
- U14 pad 1: Net-(C80-Pad2) -> /STM/temperatureADC_0/3V3_SENS
- U14 pad 10: Net-(C78-Pad1) -> Net-(U14-Pad10)
- U14 pad 2: /BATTERY MANAGER/SDA -> /STM/SDA
- U14 pad 3: /BATTERY MANAGER/SCL -> /STM/SCL
- U14 pad 5: +3V3 -> /STM/temperatureADC_0/3V3_SENS
- U14 pad 6: /BATTERY MANAGER/Temperature/ADC_nINT -> /STM/ADC_nINT
- U14 pad 7: (no net) -> GND
- U14 pad 8: (no net) -> GND
- U14 pad 9: Net-(C79-Pad1) -> Net-(U14-Pad9)
- U15 pad 1: /CB0N -> +5V
- U15 pad 2: /CB1N -> GND
- U15 pad 3: /CB2N -> /STM/POWER_SENS_1
- U15 pad 4: /CB3N -> Net-(U15-Pad4)
- U15 pad 5: /CB4N -> /STM/temperatureADC_3/3V3_SENS
- U3 pad 1: Net-(J19-Pad2) -> /DCDC_80Vto5V/5V_ISO
- U3 pad 2: (no net) -> Net-(R2-Pad1)
- U3 pad 3: Net-(J19-Pad1) -> VCC
- U3 pad 4: /BATTERY MANAGER/IMB -> /DCDC_80Vto5V/EN-DCDC1
- U4 pad 1: Net-(J20-Pad2) -> /DCDC_80Vto5V/GND_SUPPLY
- U4 pad 2: (no net) -> /DCDC_80Vto5V/GND_SUPPLY
- U4 pad 3: Net-(J20-Pad1) -> VCC
- U4 pad 4: /BATTERY MANAGER/IMA -> /DCDC_80Vto5V/EN-D
- U4 pad 5: (no net) -> Net-(R5-Pad2)
- U4 pad 6: /BATTERY MANAGER/IPA -> /DCDC_80Vto5V/SS-D
- U5 pad 10: /BATTERY MANAGER/Temperature/TX -> /STM/CS_EEPROM
- U5 pad 11: /BATTERY MANAGER/Temperature/RX -> /BATTERY MANAGER/CLK
- U5 pad 12: /BATTERY MANAGER/~CS~ -> /BATTERY MANAGER/MISO
- U5 pad 13: /BATTERY MANAGER/CLK -> /BATTERY MANAGER/MOSI
- U5 pad 14: /BATTERY MANAGER/MISO -> /STM/SPI_CS
- U5 pad 15: /BATTERY MANAGER/MOSI -> /STM/~HOLD~
- U5 pad 16: /BATTERY MANAGER/Temperature/ADC_nINT -> GND
- U5 pad 17: /BATTERY MANAGER/Temperature/POWER_SENS_2 -> +3V3
- U5 pad 18: /BATTERY MANAGER/Temperature/POWER_SENS_1 -> /STM/ADC_nINT
- U5 pad 19: GND -> /STM/TX
- U5 pad 2: /BATTERY MANAGER/DRIVE -> /STM/POWER_SENS_2
- U5 pad 20: +3V3 -> /STM/RX
- U5 pad 21: +3V3 -> /STM/CAN_RX
- U5 pad 22: (no net) -> /STM/CAN_TX
- U5 pad 23: GND -> /STM/SWDIO
- U5 pad 24: +3V3 -> /STM/SWCLK
- U5 pad 25: /BATTERY MANAGER/Temperature/~HOLD~ -> Net-(R19-Pad1)
- U5 pad 26: /BATTERY MANAGER/Temperature/CS_EEPROM -> Net-(JP2-Pad2)
- U5 pad 27: /BATTERY MANAGER/Temperature/SCK_EEPROM -> /STM/MISO_EEPROM
- U5 pad 28: /BATTERY MANAGER/Temperature/MISO_EEPROM -> /STM/MOSI_EEPROM
- U5 pad 29: /BATTERY MANAGER/Temperature/MOSI_EEPROM -> /STM/SCL
- U5 pad 3: Net-(R19-Pad1) -> /STM/POWER_SENS_1
- U5 pad 30: (no net) -> /STM/SDA
- U5 pad 31: (no net) -> GND
- U5 pad 32: (no net) -> GND
- U5 pad 33: /BATTERY MANAGER/Temperature/CAN_RX -> GND
- U5 pad 4: (no net) -> /STM/RESET
- U5 pad 5: (no net) -> +3V3
- U5 pad 6: (no net) -> Net-(U21-Pad3)
- U5 pad 7: /BATTERY MANAGER/Temperature/RESET -> /STM/ADD_2
- U5 pad 8: (no net) -> /STM/ADD_1
- U5 pad 9: (no net) -> /STM/ADD_0
- U6 pad 1: Net-(C26-Pad2) -> /STM/temperatureADC_3/3V3_SENS
- U6 pad 10: Net-(C19-Pad1) -> Net-(U6-Pad10)
- U6 pad 2: /BATTERY MANAGER/SDA -> /STM/SDA
- U6 pad 3: /BATTERY MANAGER/SCL -> /STM/SCL
- U6 pad 5: +3V3 -> /STM/temperatureADC_3/3V3_SENS
- U6 pad 6: /BATTERY MANAGER/Temperature/ADC_nINT -> /STM/ADC_nINT
- U6 pad 7: +3V3 -> GND
- U6 pad 8: GND -> /STM/temperatureADC_3/A1
- U6 pad 9: Net-(C25-Pad1) -> Net-(U6-Pad9)
- U7 pad 1: Net-(C44-Pad2) -> /STM/temperatureADC_4/3V3_SENS
- U7 pad 10: Net-(C36-Pad1) -> Net-(U7-Pad10)
- U7 pad 2: /BATTERY MANAGER/SDA -> /STM/SDA
- U7 pad 3: /BATTERY MANAGER/SCL -> /STM/SCL
- U7 pad 5: +3V3 -> /STM/temperatureADC_4/3V3_SENS
- U7 pad 6: /BATTERY MANAGER/Temperature/ADC_nINT -> /STM/ADC_nINT
- U7 pad 7: GND -> /STM/temperatureADC_4/A0
- U7 pad 8: +3V3 -> /STM/temperatureADC_4/A0
- U7 pad 9: Net-(C43-Pad1) -> Net-(U7-Pad9)
- U8 pad 1: /BATTERY MANAGER/DCDC_80Vto5V/VIN -> /DCDC_80Vto5V/120V_linreg
- U8 pad 3: Net-(JP21-Pad2) -> (no net)
- U8 pad 5: (no net) -> /DCDC_80Vto5V/GND_SUPPLY
- U8 pad 6: /BATTERY MANAGER/0V -> Net-(C84-Pad1)
- U8 pad 8: /BATTERY MANAGER/DCDC_80Vto5V/RT -> Net-(C84-Pad1)
- U8 pad 9: /BATTERY MANAGER/0V -> /DCDC_80Vto5V/GND_SUPPLY
- U9 pad 1: Net-(L2-Pad1) -> /STM/temperatureADC_2/3V3_SENS
- U9 pad 11: Net-(R50-Pad1) -> Net-(C41-Pad1)
- U9 pad 12: GND -> Net-(C40-Pad1)
- U9 pad 14: /BATTERY MANAGER/CB18 -> Net-(C38-Pad1)
- U9 pad 16: GND -> Net-(C36-Pad1)
- U9 pad 3: /BATTERY MANAGER/CB18 -> /STM/SCL
- U9 pad 5: (no net) -> /STM/temperatureADC_2/3V3_SENS
- U9 pad 6: GND -> /STM/ADC_nINT
- U9 pad 7: Net-(U9-Pad10) -> /STM/temperatureADC_2/3V3_SENS
- U9 pad 9: Net-(C24-Pad1) -> Net-(U9-Pad9)
Routing:
- net /CB0N: track 1185.9 -> 13.9 mm, vias 58 -> 0
- net VCC: track 0.00 -> 551.6 mm, vias 0 -> 4
- net +5V: track 345.6 -> 831.5 mm, vias 4 -> 5
- net /BATTERY MANAGER/SDA: track 454.8 -> 0.00 mm, vias 8 -> 0
- net /BATTERY MANAGER/SCL: track 452.4 -> 0.00 mm, vias 9 -> 0
- net /STM/SCL: track 0.00 -> 449.2 mm, vias 0 -> 11
- net /STM/SDA: track 0.00 -> 447.2 mm, vias 0 -> 11
- net /STM/ADC_nINT: track 0.00 -> 418.3 mm, vias 0 -> 11
- net /BATTERY MANAGER/Temperature/ADC_nINT: track 412.8 -> 0.00 mm, vias 8 -> 0
- net +3V3: track 555.1 -> 142.6 mm, vias 14 -> 5
- net /BATTERY MANAGER/Temperature/POWER_SENS_1: track 397.4 -> 0.00 mm, vias 6 -> 0
- net /BATTERY MANAGER/DRIVE: track 331.4 -> 0.00 mm, vias 3 -> 0
- net /STM/POWER_SENS_1: track 0.00 -> 322.0 mm, vias 0 -> 4
- net /BATTERY MANAGER/Temperature/POWER_SENS_2: track 258.5 -> 0.00 mm, vias 5 -> 0
- net /STM/POWER_SENS_2: track 0.00 -> 215.8 mm, vias 0 -> 9
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- added copper zone on F.Cu, net +5V
- added copper zone on B.Cu, net /DCDC_80Vto5V/GND_SUPPLY
- added copper zone on F.Cu, net /DCDC_80Vto5V/GND_SUPPLY
- added copper zone on F.Cu, net /DCDC_80Vto5V/SW-D
- added copper zone on F.Cu, net VCC
- removed copper zone on B.Cu, net /BATTERY MANAGER/0V
- removed copper zone on F.Cu, net /BATTERY MANAGER/0V
Other:
- outline, holes or cut-outs redrawn
- board text added: "+5V"
- board text added: "00"
- board text added: "01"
- board text added: "02"
- board text added: "03"
- board text added: "04"
- board text added: "05"
- board text added: "06"
- board text added: "07"
- board text added: "08"
- board text added: "09"
- board text added: "10"
- board text added: "11"
- board text added: "12"
- board text added: "13"
- board text added: "14"
- board text added: "15"
- board text added: "16"
- board text added: "17"
- board text added: "18"
- board text added: "20210614"
- board text added: "3"
- board text added: "3V3"
- board text added: "4"
- board text added: "5"
- board text added: "6"
- board text added: "A0"
- board text added: "A1"
- board text added: "A2"
- board text added: "C_H"
- board text added: "C_L"
- board text added: "Fenice - BMS CELLBOARD"
- board text added: "If you are reading this something went wrong, I hope it's nothing bad. Are your shoes still on?"
- board text added: "JLCJLCJLC"
- board text added: "JMP"
- board text added: "RST"
- board text added: "RX"
- board text added: "SWD"
- board text added: "SWK"
- board text added: "SWO"
- board text added: "Stencil size"
- board text added: "TX"
- board text added: "V2.1.2.5"
- board text removed: "2021"
- board text removed: "5V"
- board text removed: "BATT0"
- board text removed: "BATT1"
- board text removed: "BATT10"
- board text removed: "BATT11"
- board text removed: "BATT12"
- board text removed: "BATT13"
- board text removed: "BATT14"
- board text removed: "BATT15"
- board text removed: "BATT16"
- board text removed: "BATT17"
- board text removed: "BATT2"
- board text removed: "BATT3"
- board text removed: "BATT4"
- board text removed: "BATT5"
- board text removed: "BATT6"
- board text removed: "BATT7"
- board text removed: "BATT8"
- board text removed: "BATT9"
- board text removed: "CELL BOARD"
- board text removed: "ONLY ONE"
- board text removed: "V2.1.2.4"
