File: cellboard/CellsBoard.kicad_pcb (KiCad board)
At the start: 2 copper layers, 445.5 x 71.5 mm, 275 parts, among them CN1 10nF_array, CN2 10nF_array, CN3 10nF_array, CN4 10nF_array, CN5 10nF_array, J1 Conn_02x02_Odd_Even, J10 BUS, J11 Conn_02x06_Top_Bottom, J12 Conn_02x06_Top_Bottom, J13 Conn_02x06_Top_Bottom, J14 Conn_02x06_Top_Bottom, J15 Conn_02x06_Top_Bottom, J16 Conn_02x06_Top_Bottom, J2 Conn_02x02_Odd_Even, J3 Conn_02x02_Odd_Even, J4 Conn_02x02_Odd_Even, J5 Conn_02x02_Odd_Even, J6 Conn_02x02_Odd_Even, J7 Conn_02x05_Top_Bottom, J8 Conn_02x02_Counter_Clockwise, J9 BUS, Q1 TSM3401CX RFG, Q10 TSM3401CX RFG, Q11 TSM3401CX RFG, Q12 TSM3401CX RFG, Q13 TSM3401CX RFG, Q14 TSM3401CX RFG, Q15 BSS308PE, Q16 BSS308PE, Q17 BSS308PE, Q18 BSS308PE, Q2 TSM3401CX RFG, Q3 TSM3401CX RFG, Q4 TSM3401CX RFG, Q5 TSM3401CX RFG, Q6 TSM3401CX RFG, Q7 TSM3401CX RFG, Q8 TSM3401CX RFG, Q9 TSM3401CX RFG, SW1 RESET, U1 LTC6813-1, U10 M95256-W, U11 MAX14878AWA+, U12 ADC128D818, U13 ADC128D818, U14 ADC128D818, U15 MCP1811AT-033LT, U16 MCP1811AT-033LT, U17 MCP1811AT-033LT, U18 MCP1811AT-033LT, U19 MCP1811AT-033LT, U2 MCP1812, U20 MCP1811AT-033LT, U21 DSC61XX, U3 CPC1125N, U4 LM5161PWP, U5 STM32L432KBUx, U6 ADC128D818, U7 ADC128D818, U8 MAQ5281, U9 ADC128D818

Commit message: changed footprint mcp1811
Parts:
- U15, U16, U17, U18, U19, U20: footprint Package_TO_SOT_SMD:SOT-23-5_HandSoldering -> Package_TO_SOT_SMD:SOT-353_SC-70-5
Routing:
- net +5V: track 831.5 -> 834.1 mm
- net /STM/POWER_SENS_2: track 215.8 -> 217.4 mm
- net /STM/POWER_SENS_1: track 322.0 -> 323.5 mm
- net /STM/temperatureADC_5/3V3_SENS: track 24.1 -> 24.9 mm
- net /STM/temperatureADC_4/3V3_SENS: track 23.1 -> 23.8 mm
- net /STM/temperatureADC_1/3V3_SENS: track 22.7 -> 23.4 mm
- net /STM/temperatureADC_2/3V3_SENS: track 34.2 -> 34.9 mm
- net /STM/temperatureADC_0/3V3_SENS: track 23.2 -> 23.7 mm
