File: cellboard/LTC6813-1.sch (KiCad schematic (older format))
At the start: 36 parts, among them CN1 10nF_array, CN2 10nF_array, CN3 10nF_array, CN4 10nF_array, CN5 10nF_array, J19 CONN_1X02, J20 CONN_1X02, U1 LTC6813-1, U3 HM2103, U4 HM2103

Commit message: v2.1.2.5 as printed
Commit on behalf of fran-retfie.
Parts:
- removed C8, C9: 10nF, Capacitor_SMD:C_0603_1608Metric, symbol CellsBoard:C
- removed J19, J20: CONN_1X02, CellsBoard:Molex_Micro-Fit_3.0_43650-0215_1x02_P3.00mm_Vertical, symbol Connector_Generic:Conn_01x02
- removed JP19: GND_connection, CellsBoard:I2C_JUMPER_CONNECTION, symbol CellsBoard:I2C_Jumper
- removed JP25: SPI, CellsBoard:Jumper_adafruit, symbol CellsBoard:SolderJumper_3_Open
- removed R28, R29, R30, R31: 150, Resistor_SMD:R_0603_1608Metric, symbol CellsBoard:R
- removed RN15, RN16: 0 ohm, Resistor_SMD:R_Array_Convex_2x0603, symbol Device:R_Pack02
- removed TP2: TestPoint, CellsBoard:Test_point, symbol CellsBoard:TestPoint
- removed U3, U4: HM2103, CellsBoard:HM2103, symbol CellsBoard:HM2103
- added R1: 100, Resistor_SMD:R_0603_1608Metric, symbol Device:R
- added TP5: VRef1, TestPoint:TestPoint_Pad_D1.0mm, symbol Connector:TestPoint
- added TP6: VRef2, TestPoint:TestPoint_Pad_D1.0mm, symbol Connector:TestPoint
- added TP8: V+, TestPoint:TestPoint_Pad_D1.0mm, symbol Connector:TestPoint
- added TP9: +5V, TestPoint:TestPoint_Pad_D1.0mm, symbol Connector:TestPoint
- C10: value 100nF -> 1uF; symbol CellsBoard:C -> Device:C
- C5, C6, C7: symbol CellsBoard:C -> Device:C
- JP20: symbol CellsBoard:SolderJumper_3_Open -> Jumper:SolderJumper_3_Open
- R24: value 1k4 -> 1k; symbol CellsBoard:R -> Device:R
- R25: value 604 -> 1k; symbol CellsBoard:R -> Device:R
- R26, R27: symbol CellsBoard:R -> Device:R
Connections:
- net +5V: now also TP9.1
- net CB18: no longer R27.2
- net CLK: now also U1.62 (SCK/IPA)
- net GND: now also U1.55 (ISOMD); no longer RN10.3 (R3.1)
- net V+: now also TP8.1
- net VRef1: now also TP5.1
- net VRef2: now also TP6.1
- net ~CS~: now also U1.61 (CSB/IMA)
- net Cell0 renamed C0
- net Cell1 renamed C1
- net Cell10 renamed C10
- net Cell11 renamed C11
- net Cell12 renamed C12
- net Cell13 renamed C13
- net Cell14 renamed C14
- net Cell15 renamed C15
- net Cell16 renamed C16
- net Cell17 renamed C17
- net Cell18 renamed C18
- net Cell2 renamed C2
- net Cell3 renamed C3
- net Cell4 renamed C4
- net Cell5 renamed C5
- net Cell6 renamed C6
- net Cell7 renamed C7
- net Cell8 renamed C8
- net Cell9 renamed C9
- net DRIVE: no longer names the net of U1.49 (DRIVE)
- net IMB: no longer names the net of U1.63 (IMB)
- net IMB: now also R1.1
- net IPB: no longer names the net of U1.64 (IPB)
- net IPB: now also R1.2
- net SCL: no longer names the net of U1.42 (GPIO4)
- net SDA: no longer names the net of U1.43 (GPIO5)
- new net CB0: RN10.3 (R3.1)
- new net VCC: R27.2
- no-connect marks 11 -> 10
Other:
- note added: "C0 : Cell 1 negative sense\nCn : Cell n positive sense\nSn : Cell n balance control\nCB0 : Cell 1 negative sensing lead\nCBn : Cell n positive sensing lead"
- note removed: "If SPI is needed RN15 populated instead of RN16"
- note removed: "isoSPI_A"
- note removed: "isoSPI_B"
- moved on the sheet: C10, C5, C6, C7, JP20, S1, U1
