File: cellboard/PowerSupply.sch (KiCad schematic (older format))
At the start: 24 parts, among them J8 CONN_1X02, T40 TestPoint, U8 LT8630, U9 LTC3639

Commit message: v2.1.2.5 as printed
Commit on behalf of fran-retfie.
Parts:
- removed C23, C37: 4.7uF, Capacitor_SMD:C_1210_3225Metric, symbol CellsBoard:C
- removed C24, C41: 22uF, Capacitor_SMD:C_1210_3225Metric, symbol CellsBoard:C
- removed C38: 100pF, Capacitor_SMD:C_0603_1608Metric, symbol CellsBoard:C
- removed C39: 2.2uF, Capacitor_SMD:C_0603_1608Metric, symbol CellsBoard:C
- removed C40: 10pF, Capacitor_SMD:C_0603_1608Metric, symbol CellsBoard:C
- removed C42: 100nF_HV, Capacitor_SMD:C_1206_3216Metric, symbol CellsBoard:C
- removed D1: BAS16J, Diode_SMD:D_SOD-323, symbol CellsBoard:D
- removed F20: Fuse, CellsBoard:Fuse_0805, symbol CellsBoard:Fuse
- removed J8: CONN_1X02, CellsBoard:Molex_Micro-Fit_3.0_43650-0215_1x02_P3.00mm_Vertical, symbol Connector_Generic:Conn_01x02
- removed JP21: SolderJumper_3_Open, CellsBoard:PinHeader_1x03_P2.54mm_Vertical, symbol CellsBoard:SolderJumper_3_Open
- removed L1: 22uH, CellsBoard:SLF10145_Type_BigPad, symbol CellsBoard:L
- removed L2: 560uH, CellsBoard:Inductor_Bourns_SRR4028, symbol CellsBoard:L
- removed R20: 100, Resistor_SMD:R_0805_2012Metric, symbol CellsBoard:R
- removed R21: 25K5, Resistor_SMD:R_0603_1608Metric, symbol CellsBoard:R
- removed R22, R50: 1M, Resistor_SMD:R_0603_1608Metric, symbol CellsBoard:R
- removed R23: 191k, Resistor_SMD:R_0603_1608Metric, symbol CellsBoard:R
- removed T40, TP1, TP5: TestPoint, CellsBoard:Test_point, symbol CellsBoard:TestPoint
- removed U8: LT8630, CellsBoard:LT8631, symbol CellsBoard:LT8630
- removed U9: LTC3639, CellsBoard:MSOP-12-16-1EP_3x4mm_P0.5mm_EP1.65x2.85mm_ThermalVias, symbol CellsBoard:LTC3639
- added C1, C2, C4: 1u_HV, Capacitor_SMD:C_2220_5650Metric_Pad1.97x5.40mm_HandSolder, symbol Device:C
- added C11, C13: 10n, Capacitor_SMD:C_0805_2012Metric_Pad1.18x1.45mm_HandSolder, symbol Device:C
- added C12: 1u, Capacitor_SMD:C_0805_2012Metric_Pad1.18x1.45mm_HandSolder, symbol Device:C
- added C14: 3n, Capacitor_SMD:C_0805_2012Metric_Pad1.18x1.45mm_HandSolder, symbol Device:C
- added C15: 47u, Capacitor_SMD:C_1210_3225Metric_Pad1.33x2.70mm_HandSolder, symbol Device:C
- added C3: 100n, Capacitor_SMD:C_0805_2012Metric, symbol Device:C
- added C8: 22n, Capacitor_SMD:C_0603_1608Metric_Pad1.08x0.95mm_HandSolder, symbol Device:C
- added C9: 10n, Capacitor_SMD:C_0805_2012Metric, symbol Device:C
- added J7: Conn_02x02_Counter_Clockwise, Connector_Molex:Molex_Micro-Fit_3.0_43045-0412_2x02_P3.00mm_Vertical, symbol Connector_Generic:Conn_02x02_Counter_Clockwise
- added JP1: SolderJumper_2_Open, Jumper:SolderJumper-2_P1.3mm_Open_RoundedPad1.0x1.5mm, symbol Jumper:SolderJumper_2_Open
- added L1: 56u, CellsBoard:sdr1307, symbol Device:L
- added R2: 1.24k, Resistor_SMD:R_0805_2012Metric_Pad1.20x1.40mm_HandSolder, symbol Device:R
- added R3: 100k, Resistor_SMD:R_0805_2012Metric_Pad1.20x1.40mm_HandSolder, symbol Device:R
- added R4: 2k, Resistor_SMD:R_0805_2012Metric_Pad1.20x1.40mm_HandSolder, symbol Device:R
- added R5: 215k, Resistor_SMD:R_0805_2012Metric_Pad1.20x1.40mm_HandSolder, symbol Device:R
- added R6: 255k, Resistor_SMD:R_0805_2012Metric_Pad1.20x1.40mm_HandSolder, symbol Device:R
- added R7: 3k, Resistor_SMD:R_0603_1608Metric_Pad0.98x0.95mm_HandSolder, symbol Device:R
- added R8: 2k, Resistor_SMD:R_0603_1608Metric_Pad0.98x0.95mm_HandSolder, symbol Device:R
- added U2: CPC1125N, Package_SO:SOP-4_3.8x4.1mm_P2.54mm, symbol Relay_SolidState:CPC1117N
- added U4: LM5161PWP, Package_SO:HTSSOP-14-1EP_4.4x5mm_P0.65mm_EP3.4x5mm_Mask3x3.1mm, symbol CellsBoard:LM5161PWP
- added U8: MAQ5281, Package_SO:MSOP-8-1EP_3x3mm_P0.65mm_EP1.68x1.88mm, symbol CellsBoard:MAQ5281
Connections:
- net +5V: now also C14.2, C15.2, L1.2, R7.1
- new net: C13.2, C14.1, R6.1
- new net: C3.1, U8.4 (CPSRR)
- new net: C9.1, J7.1 (Pin_1), U8.6 (SNS), U8.8 (Vout)
- new net: C11.2, U4.11 (BST)
- new net: R5.2, U4.5 (RON)
- new net: JP1.1 (A), U4.8 (FPWM)
- new net: R2.1, U2.2
- new net 120V_linreg: C2.2, J7.3 (Pin_3), U8.1 (Vin)
- new net 5V_ISO: U2.1
- new net EN-D: R3.1, R4.2, U4.4 (EN/UVLO)
- new net EN-DCDC1: R3.2, U2.4
- new net FB-D: C13.1, R7.2, R8.1, U4.9 (FB)
- new net GND_ISO: R2.2
- new net GND_SUPPLY: C1.1, C12.1, C15.1, C2.1, C3.2, C4.1, C8.1, C9.2, J7.2 (Pin_2), R4.1, R8.2, U4.1 (AGND), U4.15 (AGND), U4.2 (PGND), U8.5 (GND), U8.9 (EP)
- new net SS-D: C8.2, U4.6 (SS)
- new net SW-D: C11.1, L1.1, R6.2, U4.12 (SW), U4.13 (SW), U4.14 (NC)
- new net VCC-D: C12.2, JP1.2 (B), U4.10 (VCC)
- new net VCC_SUPPLY: C1.2, C4.2, J7.4 (Pin_4), R5.1, U2.3, U4.3 (VIN)
- no-connect marks 3 -> 0
Other:
- note added: "Buck DCDC converter - 80V in - 5V 1A out"
- note added: "Close JP5 to enable \nCCM at light loads."
- note added: "DCDC is enabled by an optocoupled \nactivated by 5V from CAN connector"
- note added: "Disconnecting the mainboard\ndisconnects the linreg"
- note added: "EN: \n<0.35V SHUTDOWN state\n<1.24V STAND-BY state\nEN-D:\nLOW Voltage 3.5V*18cells=63V\n"
- note added: "Linear regulator 5V - 25mA"
- note added: "Populate only on segment 0"
- note removed: "2.2/4.7=(1-x)-> x=53.2%>50%"
- note removed: "ACTIVE mode\nSTM32G474-> runMODE_35mA+25mA driving\nLTC6813-1 ->16.5mA+1.1mA(ibias)+11mA (isoPSI)\nTOT:90mA (max Power require from all electtonic)"
- note removed: "Note that even X5R and X7R type ceramic capacitors have\na DC bias effect which reduces their capacitance when a\nDC voltage is applied. It is not uncommon for capacitors\noffered in the smallest case sizes to lose more than 50%\nof their capacitance when operated near their rated voltage"
- note removed: "POWER SUPPLY"
- note removed: "POWER SUPPLY FOR COCKPIT LED"
- note removed: "SLEEP mode\nSTM32G474-> standbyMODE_7.2uA\nLTC6813-1 ->6uA+0mA(ibias)+9uA (isoPSI)\nTOT:22uA (max Power require from all electtonic)"
