File: cellboard/temperatureADC.sch (KiCad schematic (older format))
At the start: 17 parts, among them J1 Conn_02x08, Q19 TSM3401CX RFG, U6 ADC128D818

Commit message: v2.1.2.5 as printed
Commit on behalf of fran-retfie.
Parts:
- removed C19, C25: 100nF, Capacitor_SMD:C_0603_1608Metric, symbol CellsBoard:C
- removed J1: Conn_02x08, CellsBoard:Molex_Micro-Fit_3.0_43045-1612_2x08_P3.00mm_Vertical, symbol CellsBoard:Conn_02x08
- removed Q19: TSM3401CX RFG, CellsBoard:SOT-23, symbol CellsBoard:Q_PMOS_GDS
- added J16: Conn_02x06_Top_Bottom, Connector_Molex:Molex_Nano-Fit_105310-xx12_2x06_P2.50mm_Vertical, symbol Connector_Generic:Conn_02x06_Top_Bottom
- added U20: MCP1811AT-033LT, Package_TO_SOT_SMD:SOT-23-5_HandSoldering, symbol CellsBoard:MCP1811AT-033LT
- C11, C14, C15, C16, C17, C18, C26, C27, C28, C29: symbol CellsBoard:C -> Device:C
- RN11, RN14: value 3K3 -> x; footprint Resistor_SMD:R_Array_Convex_4x1206 -> Resistor_SMD:R_Array_Convex_4x0603
Connections:
- net GND: now also RN14.4 (R4.1), J16.1 (Pin_1), J16.2 (Pin_2), J16.3 (Pin_3), J16.4 (Pin_4), J16.5 (Pin_5), J16.6 (Pin_6), U20.2 (GND)
- net SENS_POWER: now also U20.3 (SDWN)
- net 3V3_SENS: now reaches C26.2, C27.2, RN11.1 (R1.1), RN11.2 (R2.1), RN11.3 (R3.1), RN11.4 (R4.1), RN14.1 (R1.1), RN14.2 (R2.1), RN14.3 (R3.1), U6.1 (VREF)
- net 3V3_SENS: now also U6.5 (V+), U20.5 (Vout); no longer RN14.4 (R4.1)
- net at C14.1, U6.15 (IN1): now also RN11.7 (R2.2), J16.11 (Pin_11); no longer RN11.6 (R3.2)
- net at C15.1, U6.14 (IN2): now also RN11.6 (R3.2), J16.10 (Pin_10); no longer RN11.7 (R2.2)
- net at C16.1, U6.13 (IN3): now also RN11.5 (R4.2), J16.9 (Pin_9); no longer RN11.8 (R1.2)
- net at C17.1, U6.12 (IN4): now also RN14.8 (R1.2), J16.8 (Pin_8); no longer RN14.5 (R4.2)
- net at C18.1, U6.11 (IN5): now also RN14.7 (R2.2), J16.7 (Pin_7); no longer RN14.6 (R3.2)
- net at U6.10 (IN6): no longer RN14.7 (R2.2)
- net at U6.9 (IN7): no longer RN14.8 (R1.2)
- net at C11.1, U6.16 (IN0): now also RN11.8 (R1.2), J16.12 (Pin_12); no longer RN11.5 (R4.2)
- net +3V3 renamed +5V
- net +5V: now also U20.1 (Vin); no longer U6.5 (V+)
- net SCL1 renamed SCL
- net SDA1 renamed SDA
- new net MID: RN14.5 (R4.2), RN14.6 (R3.2)
- no-connect marks 0 -> 3
Other:
- moved on the sheet: C28, C29
