File: mainboard/MCU.sch (KiCad schematic (older format))
At the start: 64 parts, among them J9 Micro_SD_Card_Det_Hirose_DM3AT, SW1 RESET, U11 STM32G474, U12 M95256-WMN6P, U17 CD74HC4067SM, U5 MCP2562, U6 LM358, U8 LTC6820, U9 HM2103

Commit message: Corrected BOOT0
Other:
- note added: "PB8-BOOT0 pin configuration:\nLOW: normal, boot from user flash\nHIGH: boot from system memory, bootloader"
- note removed: "Switch this and BOOT0 so to have it work"
Changed lines of the file:
@@
 Text Label 8850 700  3    50   ~ 0
 CAN_TX
-Text Label 8950 700  3    50   ~ 0
+Text Label 10450 1700 2    50   ~ 0
 CAN_RX
 Wire Wire Line
@@
 	9450 1000 9450 1050
 Wire Wire Line
-	8950 1050 8950 700
+	10100 1700 10450 1700
 Wire Wire Line
 	9250 1000 9250 1050
@@
 Wire Wire Line
 	10100 2400 11200 2400
-Text HLabel 10100 1700 2    50   Input ~ 0
+Text HLabel 8950 1050 1    50   Input ~ 0
 PC_ENDED
 Text HLabel 10100 1800 2    50   Input ~ 0
@@
 Wire Wire Line
 	6600 6600 6600 6400
+Text Label 6500 6400 3    50   ~ 0
+A2
 Text Label 6700 6400 3    50   ~ 0
-A2
-Text Label 6500 6400 3    50   ~ 0
 A0
 Wire Wire Line
-	6500 6400 6500 6600
-Wire Wire Line
-	6700 6600 6700 6400
+	6700 6400 6700 6600
+Wire Wire Line
+	6500 6600 6500 6400
 Text Label 6800 6400 3    50   ~ 0
 A3
@@
 	1    0    0    -1
 $EndComp
-Text Notes 10550 1750 0    50   ~ 0
-Switch this and BOOT0 so to have it work
+Text Notes 6350 800  0    50   ~ 0
+PB8-BOOT0 pin configuration:\nLOW: normal, boot from user flash\nHIGH: boot from system memory, bootloader
 $EndSCHEMATC

Commit message: Added jumper for BOOT0 to 3V3
Parts:
- added JP4: SolderJumper_2_Open, MainBoard:Jumper_SMD_0603, symbol Jumper:SolderJumper_2_Open
Changed lines of the file:
@@
 Text Notes 6350 800  0    50   ~ 0
 PB8-BOOT0 pin configuration:\nLOW: normal, boot from user flash\nHIGH: boot from system memory, bootloader
+Text HLabel 6800 850  0    50   Input ~ 0
+PC_ENDED
+$Comp
+L power:+3.3V #PWR?
+U 1 1 5FD436DF
+P 7100 850
+AR Path="/5FD436DF" Ref="#PWR?"  Part="1"
+AR Path="/5DF398FB/5FD436DF" Ref="#PWR016"  Part="1"
+F 0 "#PWR016" H 7100 700 50  0001 C CNN
+F 1 "+3.3V" V 7100 1000 50  0000 L CNN
+F 2 "" H 7100 850 50  0001 C CNN
+F 3 "" H 7100 850 50  0001 C CNN
+	1    7100 850
+	0    1    1    0
+$EndComp
+$Comp
+L Jumper:SolderJumper_2_Open JP4
+U 1 1 5FD45CCD
+P 6950 850
+F 0 "JP4" H 6900 750 50  0000 L CNN
+F 1 "SolderJumper_2_Open" V 6995 898 50  0001 L CNN
+F 2 "MainBoard:Jumper_SMD_0603" H 6950 850 50  0001 C CNN
+F 3 "~" H 6950 850 50  0001 C CNN
+	1    6950 850
+	-1   0    0    -1
+$EndComp
 $EndSCHEMATC

Commit message: Added 64pin mcu and moved isocanspi to HV sheet
Parts:
- removed C18, C19, C21: 100nF, Capacitor_SMD:C_0603_1608Metric, symbol Device:C_Small
- removed R13: 330K, Resistor_SMD:R_0603_1608Metric, symbol Device:R
- removed R34, R35: 150, Resistor_SMD:R_0603_1608Metric, symbol Device:R
- removed R38: 604, Resistor_SMD:R_0603_1608Metric, symbol Device:R
- removed R39: 1K4, Resistor_SMD:R_0603_1608Metric, symbol Device:R
- removed U11: STM32G474, Package_QFP:LQFP-48_7x7mm_P0.5mm, symbol MainBoard:STM32G474
- removed U8: LTC6820, MainBoard:MSOP-16, symbol MainBoard:LTC6820
- removed U9: HM2103, MainBoard:HM2103, symbol MainBoard:HM2103
- added U11: STM32G474R, Package_QFP:LQFP-64_10x10mm_P0.5mm, symbol MainBoard:STM32G474R
Connections:
- net labels removed: IBIAS, ICMP, IM, IM_LV, IP, IP_LV
- wire segments 256 -> 229
- no-connect marks 12 -> 10
Other:
- note added: "CAN1 INTERFACE"
- note added: "CHECK:\nIMD_PWM: moved from PA12 to PA10, ask soft\nTS_ON: moved from PA10 to PB9\n"
- note added: "supply filtering and analog rail"
- note removed: "CAN INTERFACE"
- note removed: "isoSPI INTERFACE"
- note removed: "selectable between can and spi"
- note removed: "supply filtering for analog rail"
- moved on the sheet: C13, C14, C15, C20, C22, C25, FB1, JP4, SW1

Commit message: docs
Connections:
- net A0: now also RN10.5 (R4.2), U17.10 (S0); no longer RN10.7 (R2.2), U17.14 (S2)
- net A2: now also RN10.7 (R2.2), U17.14 (S2); no longer RN10.5 (R4.2), U17.10 (S0)
Other:
- note added: "AMS: Automatic Moaning System"
- note removed: "CHECK:\nIMD_PWM: moved from PA12 to PA10, ask soft\nTS_ON: moved from PA10 to PB9\n"
- moved on the sheet: RN10
Changed lines of the file:
@@
 L Device:R_Pack04 RN?
 U 1 1 5F5FCEBB
-P 6600 6800
+P 6350 7300
 AR Path="/5B045B0D/5F5FCEBB" Ref="RN?"  Part="1"
 AR Path="/5DF398FB/5F5FCEBB" Ref="RN10"  Part="1"
-F 0 "RN10" H 6788 6846 50  0000 L CNN
-F 1 "100K" H 6788 6755 50  0000 L CNN
-F 2 "MainBoard:R_network_4x1_bourns_CAY16" V 6875 6800 50  0001 C CNN
-F 3 "https://www.mouser.it/ProductDetail/Bourns/CAY16-104J4LF?qs=sGAEpiMZZMvrmc6UYKmaNeZNuQlTB3CaDlLE%2FtUkIfI%3D" H 6600 6800 50  0001 C CNN
-F 4 "https://www.mouser.it/ProductDetail/Bourns/CAY16-104J4LF?qs=sGAEpiMZZMvrmc6UYKmaNeZNuQlTB3CaDlLE%2FtUkIfI%3D" H 6600 6800 50  0001 C CNN "Mouser"
-	1    6600 6800
+F 0 "RN10" H 6538 7346 50  0000 L CNN
+F 1 "100K" H 6538 7255 50  0000 L CNN
+F 2 "MainBoard:R_network_4x1_bourns_CAY16" V 6625 7300 50  0001 C CNN
+F 3 "https://www.mouser.it/ProductDetail/Bourns/CAY16-104J4LF?qs=sGAEpiMZZMvrmc6UYKmaNeZNuQlTB3CaDlLE%2FtUkIfI%3D" H 6350 7300 50  0001 C CNN
+F 4 "https://www.mouser.it/ProductDetail/Bourns/CAY16-104J4LF?qs=sGAEpiMZZMvrmc6UYKmaNeZNuQlTB3CaDlLE%2FtUkIfI%3D" H 6350 7300 50  0001 C CNN "Mouser"
+	1    6350 7300
 	-1   0    0    -1
 $EndComp
@@
 L power:GND #PWR?
 U 1 1 5F602093
-P 6650 7100
+P 6400 7600
 AR Path="/5F602093" Ref="#PWR?"  Part="1"
 AR Path="/5DF398FB/5F602093" Ref="#PWR0241"  Part="1"
-F 0 "#PWR0241" H 6650 6850 50  0001 C CNN
-F 1 "GND" V 6650 6950 50  0000 R CNN
-F 2 "" H 6650 7100 50  0001 C CNN
-F 3 "" H 6650 7100 50  0001 C CNN
-	1    6650 7100
-	1    0    0    -1
-$EndComp
-Wire Wire Line
-	6500 7050 6500 7000
-Wire Wire Line
-	6800 7050 6800 7000
-Wire Wire Line
-	6500 7050 6600 7050
-Wire Wire Line
-	6650 7100 6650 7050
-Connection ~ 6650 7050
-Wire Wire Line
-	6650 7050 6700 7050
-Wire Wire Line
-	6600 7000 6600 7050
-Connection ~ 6600 7050
-Wire Wire Line
-	6600 7050 6650 7050
-Wire Wire Line
-	6700 7000 6700 7050
-Connection ~ 6700 7050
-Wire Wire Line
-	6700 7050 6800 7050
-Text Label 6600 6400 3    50   ~ 0
-A1
-Wire Wire Line
-	6600 6600 6600 6400
-Text Label 6500 6400 3    50   ~ 0
-A2
-Text Label 6700 6400 3    50   ~ 0
-A0
-Wire Wire Line
-	6700 6400 6700 6600
-Wire Wire Line
-	6500 6600 6500 6400
-Text Label 6800 6400 3    50   ~ 0
-A3
-Wire Wire Line
-	6800 6600 6800 6400
+F 0 "#PWR0241" H 6400 7350 50  0001 C CNN
+F 1 "GND" H 6400 7450 50  0000 C CNN
+F 2 "" H 6400 7600 50  0001 C CNN
+F 3 "" H 6400 7600 50  0001 C CNN
+	1    6400 7600
+	1    0    0    -1
+$EndComp
+Wire Wire Line
+	6250 7550 6250 7500
+Wire Wire Line
+	6550 7550 6550 7500
+Wire Wire Line
+	6250 7550 6350 7550
+Wire Wire Line
+	6400 7600 6400 7550
+Connection ~ 6400 7550
+Wire Wire Line
+	6400 7550 6450 7550
+Wire Wire Line
+	6350 7500 6350 7550
+Connection ~ 6350 7550
+Wire Wire Line
+	6350 7550 6400 7550
+Wire Wire Line
+	6450 7500 6450 7550
+Connection ~ 6450 7550
+Wire Wire Line
+	6450 7550 6550 7550
 Text Label 3900 7550 0    50   ~ 0
 CHECK_MUX
@@
 	-1   0    0    -1
 $EndComp
-Text Label 5850 6750 2    50   ~ 0
+Text Label 6850 6750 2    50   ~ 0
 A1
-Wire Wire Line
-	5650 6750 5850 6750
-Text Label 5850 6650 2    50   ~ 0
+Text Label 6850 6850 2    50   ~ 0
 A2
-Text Label 5850 6850 2    50   ~ 0
+Text Label 6850 6650 2    50   ~ 0
 A0
-Wire Wire Line
-	5850 6650 5650 6650
-Wire Wire Line
-	5650 6850 5850 6850
-Text Label 5850 6950 2    50   ~ 0
+Text Label 6850 6950 2    50   ~ 0
 A3
-Wire Wire Line
-	5650 6950 5850 6950
 Wire Wire Line
 	4650 7550 4550 7550
@@
 Text HLabel 7600 2550 0    50   Input ~ 0
 NRST
-Text Notes 7650 750  0    50   ~ 0
-CHECK:\nIMD_PWM: moved from PA12 to PA10, ask soft\nTS_ON: moved from PA10 to PB9\n
 Text Label 10450 3350 2    50   ~ 0
 CS_CARD
@@
 Text HLabel 8450 3900 3    50   Input ~ 0
 MOSI
+Wire Wire Line
+	5650 6650 6250 6650
+Wire Wire Line
+	5650 6750 6350 6750
+Wire Wire Line
+	5650 6850 6450 6850
+Wire Wire Line
+	5650 6950 6550 6950
+Wire Wire Line
+	6550 7100 6550 6950
+Connection ~ 6550 6950
+Wire Wire Line
+	6550 6950 6850 6950
+Wire Wire Line
+	6450 7100 6450 6850
+Connection ~ 6450 6850
+Wire Wire Line
+	6450 6850 6850 6850
+Wire Wire Line
+	6350 7100 6350 6750
+Connection ~ 6350 6750
+Wire Wire Line
+	6350 6750 6850 6750
+Wire Wire Line
+	6250 7100 6250 6650
+Connection ~ 6250 6650
+Wire Wire Line
+	6250 6650 6850 6650
+Text Notes 7000 6650 0    50   ~ 0
+AMS: Automatic Moaning System
 $EndSCHEMATC
