File: mainboard/MCU.sch (KiCad schematic (older format))
At the start: 49 parts, among them J12 SPARE_PINS, J9 Micro_SD_Card_Det_Hirose_DM3AT, SW1 RESET, U12 M95256-WMN6P, U5 MCP2562, U6 LM358, U9 STM32F446RE_64PIN, Y1 16MHz

Commit message: Correction almost finished, Started layouting
Parts:
- removed unit 2 of RN14
- removed unit 1 of RN14
- removed unit 4 of RN14
- added BZ1: Buzzer, Eagle_Main:Buzzer_TDK_SD1614TT_D16mm_H14mm_P5mm, symbol Device:Buzzer
- added D14: 1N4148W, Diode_SMD:D_SOD-123, symbol Diode:1N4148W
- added J1: CONN_1x4, Connector_Molex:Molex_Micro-Fit_3.0_43650-0415_1x04_P3.00mm_Vertical, symbol Connector_Generic:Conn_01x04
- added Q1, Q8: 2N7002NXAKR, Package_TO_SOT_SMD:SOT-23, symbol Transistor_FET:2N7002
- added R35: 120, Resistor_SMD:R_0805_2012Metric, symbol Device:R
- added R37, R4: 10K, Resistor_SMD:R_0603_1608Metric, symbol Device:R
- added RN19: 22, Resistor_SMD:R_Array_Convex_4x0603, symbol Device:R_Pack04_Split
- added RN27: 22, Resistor_SMD:R_Array_Convex_4x0603, symbol Device:R_Pack04
- D8: footprint MainBoard:LED_REVERSE_MOUNT_cilindrical -> Eagle_Main:LED_reverse_mount_cilindrical
- JP1: renamed from B-H1; footprint MainBoard:Jumper_SMD_0603 -> Jumper:SolderJumper-2_P1.3mm_Open_RoundedPad1.0x1.5mm
- RN1, RN12, RN22, RN9: footprint MainBoard:R_network_4x1_bourns_CAY16 -> Resistor_SMD:R_Array_Convex_4x0603
- RN14: footprint MainBoard:R_network_4x1_bourns_CAY16 -> Resistor_SMD:R_Array_Convex_4x0603; symbol Device:R_Pack04_Split -> Device:R_Pack04
- SW1: footprint MainBoard:Button_SMD_6x3.5x4.3mm -> Button_Switch_SMD:SW_SPST_FSMSM; symbol MainBoard:SW_Push -> Switch:SW_Push
- U12: symbol MainBoard:M95M56-WMN6P -> Memory_EEPROM:M95256-WMN6P
- U5: symbol MainBoard:MCP2562 -> Interface_CAN_LIN:MCP2562-E-SN
- U9: symbol MainBoard:STM32F446RE_64PIN -> Eagle_Main:STM32F446RETx_physical
Connections:
- net MISO_2 is gone; now on net SPI2_MISO: J9.7 (DAT0), U12.2 (Q)
- net MOSI_2 is gone; now on net SPI2_MOSI: J9.3 (CMD), U12.5 (D)
- net +3V3: no longer R6.1
- net +5V: now also R6.1, BZ1.1 (-), D14.1 (K), J1.4 (Pin_4)
- net CAN+: now also R35.1
- net CAN-: now also R35.2
- net GND: now also J1.2 (Pin_2), Q1.2 (S), Q8.2 (S)
- net HIGH_CURRENT: now also J1.3 (Pin_3)
- net LOW_CURRENT: now also J1.1 (Pin_1)
- net MUX_A0: no longer U9.21 (PA5/SPI1SCK)
- net MUX_A1: no longer U9.22 (PA6/SPI1MISO)
- net MUX_A2: no longer U9.23 (PA7/SPI1MOSI)
- net MUX_A3: no longer U9.24 (PC4)
- net PB7: no longer U9.59 (PB7/I2C_1SDA)
- net SCK_2: no longer J9.5 (CLK), RN14.6 (R3.2), U12.6 (C)
- net SPI2_MISO: now also RN14.2 (R2.1); no longer R6.2, U9.35 (PB14)
- net SPI2_MOSI: now also RN14.1 (R1.1); no longer U9.36 (PB15)
- net SPI2_SCK: now also J9.5 (CLK), U12.6 (C); no longer U9.34 (PB13)
- net at R22.2, U6.7: now also R37.1; no longer U6.6 (-)
- net at R17.2, U6.1: now also R4.1; no longer U6.2 (-)
- net ADC_RX: no longer names the net of U9.25 (PC5)
- net ADC_SIN: no longer names the net of U9.26 (PB0)
- net ADC_SIN: no longer RN12.8 (R1.2)
- net ADC_TX: no longer names the net of U9.29 (PB10)
- net CARD_OK renamed CARD_DET
- net FB_FROM_TSMS renamed FB_SD_END
- net FB_RELAY_LV renamed FB_SD_RELAY_D
- new net: R4.2, U6.2 (-)
- new net: R37.2, U6.6 (-)
- new net: Q8.1 (G), RN19.1 (R1.1)
- new net: BZ1.2 (+), D14.2 (A), Q1.3 (D)
- new net: Q1.1 (G), RN19.2 (R2.1)
- new net BUZZER: RN19.7 (R2.2)
- new net CS_ADC: RN27.4 (R4.1)
- new net CS_ADC_: RN27.5 (R4.2), U9.24 (PC4)
- new net FAN_PWM: Q8.3 (D), R6.2
- new net FAN_PWM_N: RN12.8 (R1.2), RN19.8 (R1.2), U9.59 (PB7/I2C_1SDA)
- new net SPI1_MISO: RN27.2 (R2.1)
- new net SPI1_MISO_: RN27.7 (R2.2), U9.22 (PA6/SPI1MISO)
- new net SPI1_MOSI: RN27.3 (R3.1)
- new net SPI1_MOSI_: RN27.6 (R3.2), U9.23 (PA7/SPI1MOSI)
- new net SPI1_SCK: RN27.1 (R1.1)
- new net SPI1_SCK_: RN27.8 (R1.2), U9.21 (PA5/SPI1SCK)
- new net SPI2_MISO_: RN14.7 (R2.2), U9.35 (PB14)
- new net SPI2_MOSI_: RN14.6 (R3.2), U9.36 (PB15)
- new net SPI2_SCK_: RN14.8 (R1.2), U9.34 (PB13)
- no-connect marks 6 -> 8
Other:
- note added: "BUZZER"
- note added: "DHAB S/160"
- note added: "DNP"
- note added: "FANS"
- note added: "HALL CURRENT SENSOR"
- note added: "RC filter fc=60kHz"
- note added: "SPI MEMORIES"
- note removed: "AMS: Accumulator Management System"
- note removed: "BUFFERED CURRENT SENSOR"
- note removed: "SPI ROM"
- note removed: "microSD CARD"
- moved on the sheet: C10, C11, C12, C22, C30, C6, C7, C8, C9, D10, D8, D9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
