File: mainboard/MainBoard.kicad_pcb (KiCad board)
At the start: 2 copper layers, 155 x 73.2 mm, 249 parts, among them J1 CONN_1x4, J10 AIR+, J11 CONN_2X2, J12 SPARE_PINS, J17 HV, J18 CONN_1X2, J19 CONN_1X2, J2 CONN_2X3, J3 CONN_2X3, J4 CONN_2X2, J5 SWDEBUG_CONNECTOR, J6 AIR-, J7 CONN_2X12, J8 CONN_1X2, J9 Micro_SD_Card_Det_Hirose_DM3AT, K1 KT12-1A, K2 G6DN 12V, Q1 NTR5105PT1G, Q10 NTR5105PT1G, Q11 NTR5105PT1G, Q12 NTR5105PT1G, Q2 DMN10H220L, Q3 DMN10H220L, Q4 2N7002NXAKR, Q5 2N7002NXAKR, Q6 2N7002NXAKR, Q7 DMN10H220L, Q8 NTR5105PT1G, Q9 NTR5105PT1G, SW1 RESET, SW2 SD_RESET, U1 Tex_DCDC, U11 TS3704IPT, U12 M95256-WMN6P, U13 TS3704IPT, U14 CD4044, U15 CD4082, U16 ADCMP350, U19 TCMT1103, U2 TSC211, U24 LM358, U26 TCMT1103, U27 DCDC_ISO_5V, U28 MIC5365-3.3YC5, U29 Si8900, U30 MAX14878AWA+, U4 MainBoard_AD8244, U5 MCP2562, U6 LM358, U7 ADCMP354, U8 CD74HC4067SM, U9 STM32F446RE_64PIN, Y1 26MHz

Commit message: Correction almost finished, Started layouting
Parts:
- removed C35, C41, C47: 100nF, Capacitor_SMD:C_0603_1608Metric
- removed C43: 10nF, Capacitor_SMD:C_0603_1608Metric
- removed D20: D, MainBoard:SOD_323HE
- removed J4: CONN_2X2, MainBoard:Molex_Micro-Fit_3.0_43045-0612_2x03_P3.00mm_Vertical
- removed the JP1 at (213.7, 81.0)
- removed R29, R57: 100K, Resistor_SMD:R_0603_1608Metric
- removed R30, R31, R32, R33, R34, R39, R40: 0, Resistor_SMD:R_0603_1608Metric
- removed R54: 1M, Resistor_SMD:R_0603_1608Metric
- removed R56: 10M, Resistor_SMD:R_2010_5025Metric
- removed R59: 100, Resistor_SMD:R_0603_1608Metric
- removed R70: 680, Resistor_SMD:R_0603_1608Metric
- removed TP19: PC_ST, TestPoint:TestPoint_Pad_D1.0mm
- removed TP43: 11, TestPoint:TestPoint_Pad_D1.0mm
- removed TP44: 9, TestPoint:TestPoint_Pad_D1.0mm
- removed TP45: 13, TestPoint:TestPoint_Pad_D1.0mm
- removed TP46: 14, TestPoint:TestPoint_Pad_D1.0mm
- removed U19, U26: TCMT1103, Package_SO:SOP-4_4.4x2.6mm_P1.27mm
- removed U29: Si8900, Package_SO:SOIC-16W_7.5x10.3mm_P1.27mm
- added BZ1: Buzzer, Eagle_Main:Buzzer_TDK_SD1614TT_D16mm_H14mm_P5mm, F.Cu at (61.8, 95.0)
- added C4: 100nF, Capacitor_SMD:C_0603_1608Metric, F.Cu at (212.8, 86.8)
- added C5: 100nF, Capacitor_SMD:C_0603_1608Metric, F.Cu at (217.1, 85.0)
- added JP8: SolderJumper_2_Open, Jumper:SolderJumper-2_P1.3mm_Open_RoundedPad1.0x1.5mm, F.Cu at (180.3, 45.7)
- added Q13: DMN10H220L, Package_TO_SOT_SMD:SOT-23, F.Cu at (121.9, 55.5)
- added Q14: DMN10H220L, Package_TO_SOT_SMD:SOT-23, F.Cu at (125.4, 51.6)
- added Q15: DMN10H220L, Package_TO_SOT_SMD:SOT-23, F.Cu at (125.4, 55.5)
- added Q16: 2N7002NXAKR, Package_TO_SOT_SMD:SOT-23, F.Cu at (195.0, 58.0)
- added Q17: 2N7002NXAKR, Package_TO_SOT_SMD:SOT-23, F.Cu at (127.3, -28.2)
- added Q18: 2N7002NXAKR, Package_TO_SOT_SMD:SOT-23, F.Cu at (123.4, -28.2)
- added Q19: 2N7002NXAKR, Package_TO_SOT_SMD:SOT-23, F.Cu at (146.8, -28.2)
- added Q20: 2N7002NXAKR, Package_TO_SOT_SMD:SOT-23, F.Cu at (142.9, -28.2)
- added Q21: NTR5105PT1G, Package_TO_SOT_SMD:SOT-23, F.Cu at (142.2, -19.1)
- added R37: 10K, Resistor_SMD:R_0603_1608Metric, F.Cu at (98.3, 50.4)
- added R38: 100K, Resistor_SMD:R_0603_1608Metric, F.Cu at (124.7, 78.5)
- added R4: 10K, Resistor_SMD:R_0603_1608Metric, F.Cu at (104.2, 52.0)
- added R41: 71K5, Resistor_SMD:R_0603_1608Metric, F.Cu at (226.1, 85.7)
- added R42: 71K5, Resistor_SMD:R_0603_1608Metric, F.Cu at (226.1, 80.0)
- added RN23: 22, Resistor_SMD:R_Array_Convex_4x0603, F.Cu at (150.3, -6.59)
- added RN24: 330k, Resistor_SMD:R_Array_Convex_4x0603, F.Cu at (162.5, 0.25)
- added RN25: 22, Resistor_SMD:R_Array_Convex_4x0603, F.Cu at (184.4, 52.8)
- added RN26: 22, Resistor_SMD:R_Array_Convex_4x0603, F.Cu at (123.0, -4.86)
- added RN27: 22, Resistor_SMD:R_Array_Convex_4x0603, F.Cu at (119.2, 19.8)
- added RN28: 100K, Resistor_SMD:R_Array_Convex_4x0603, F.Cu at (141.2, -23.3)
- added TP32: EXT_LATCHED, TestPoint:TestPoint_Pad_D1.0mm, F.Cu at (179.9, -11.2)
- added U10: TCMT1103, Package_SO:SOP-4_4.4x2.6mm_P1.27mm, F.Cu at (203.0, 71.8)
- added U17: TS3704, Package_SO:TSSOP-14_4.4x5mm_P0.65mm, F.Cu at (135.8, 72.4)
- added U3: TS3702IPT, Package_SO:TSSOP-8_4.4x3mm_P0.65mm, F.Cu at (214.6, 77.1)
- C17: value 1uF -> 100nF; footprint Capacitor_SMD:C_0805_2012Metric -> Capacitor_SMD:C_0603_1608Metric
- D11, D15, D16, D17: value D -> 1N4148W; footprint MainBoard:SOD_323HE -> Diode_SMD:D_SOD-123
- D14: value DDZ13ASF 13V -> 1N4148W; footprint Diode_SMD:D_SOD-323 -> Diode_SMD:D_SOD-123
- D19: value D -> DDZ13ASF 13V; footprint MainBoard:SOD_323HE -> Diode_SMD:D_SOD-323
- D4: value LED_Small -> TS_OFF
- D8: footprint MainBoard:LED_REVERSE_MOUNT_cilindrical -> Eagle_Main:LED_reverse_mount_cilindrical
- G***: footprint MainBoard:logo_21.2mm -> Eagle_Logos:logo_21.2mm
- G***: footprint MainBoard:logo_40mm -> Eagle_Logos:logo_40mm
- G***: footprint MainBoard:scritta_scale500 -> Eagle_Logos:scritta_scale500
- H1, H2, H3, H4, H5: footprint MountingHole:MountingHole_3mm -> Eagle_Main:MountingHole_3.2_6.1Free
- J1: footprint MainBoard:Molex_Micro-Fit_3.0_43650-0415_1x04_P3.00mm_Vertical -> Connector_Molex:Molex_Micro-Fit_3.0_43650-0415_1x04_P3.00mm_Vertical
- J10, J6: footprint MainBoard:Molex_Micro-Fit_3.0_43045-0412_2x02_P3.00mm_Vertical -> Connector_Molex:Molex_Micro-Fit_3.0_43045-0412_2x02_P3.00mm_Vertical
- J11: value CONN_2X2 -> isoCAN; footprint MainBoard:Molex_Micro-Fit_3.0_43045-0412_2x02_P3.00mm_Vertical -> Connector_Molex:Molex_Micro-Fit_3.0_43045-0412_2x02_P3.00mm_Vertical
- J17: footprint MainBoard:Molex_Mega-Fit_76829-0104_2x02_P5.70mm_Vertical -> Connector_Molex:Molex_Mega-Fit_76829-0104_2x02_P5.70mm_Vertical
- J18: value CONN_1X2 -> IMD_TS+; footprint MainBoard:Molex_Micro-Fit_3.0_43650-0215_1x02_P3.00mm_Vertical -> Connector_Molex:Molex_Micro-Fit_3.0_43650-0215_1x02_P3.00mm_Vertical
- J19: value CONN_1X2 -> IMD_TS-; footprint MainBoard:Molex_Micro-Fit_3.0_43650-0215_1x02_P3.00mm_Vertical -> Connector_Molex:Molex_Micro-Fit_3.0_43650-0215_1x02_P3.00mm_Vertical
- J2: value CONN_2X3 -> CAN_POWER; footprint MainBoard:Molex_Micro-Fit_3.0_43045-0612_2x03_P3.00mm_Vertical -> Connector_Molex:Molex_Micro-Fit_3.0_43045-0612_2x03_P3.00mm_Vertical
- J3: footprint MainBoard:Molex_Micro-Fit_3.0_43045-0612_2x03_P3.00mm_Vertical -> Connector_Molex:Molex_Micro-Fit_3.0_43045-0612_2x03_P3.00mm_Vertical
- J7: value CONN_2X12 -> SIGNALS_INOUT; footprint MainBoard:Molex_Micro-Fit_3.0_43045-1212_2x06_P3.00mm_Vertical -> Connector_Molex:Molex_Micro-Fit_3.0_43045-1212_2x06_P3.00mm_Vertical
- J8: footprint MainBoard:Molex_Micro-Fit_3.0_43650-0215_1x02_P3.00mm_Vertical -> Connector_Molex:Molex_Micro-Fit_3.0_43650-0215_1x02_P3.00mm_Vertical
- JP1: renamed from B-H1; footprint MainBoard:Jumper_SMD_0603 -> Jumper:SolderJumper-2_P1.3mm_Open_RoundedPad1.0x1.5mm
- K1: footprint MainBoard:KT_THT -> Eagle_Main:KT12_THT
- K2: value G6DN 12V -> OJE-SH-112DM; footprint MainBoard:G6DN-1A_DC12 -> Eagle_Main:OJE-SH-112DM
- Q1, Q10, Q11, Q8, Q9: value NTR5105PT1G -> 2N7002NXAKR
- Q3, Q7: value DMN10H220L -> DMN10H220LK3; footprint Package_TO_SOT_SMD:SOT-23 -> Package_TO_SOT_SMD:TO-252-2
- Q5, Q6: value 2N7002NXAKR -> 2N7002NXAKR
- R16: value 1K -> 10M 1%; footprint Resistor_SMD:R_0603_1608Metric -> Resistor_SMD:R_2010_5025Metric
- R19, R21: value 1K -> 270k 10%
- R20: value 0 -> 10M; footprint Resistor_SMD:R_0603_1608Metric -> Resistor_SMD:R_2010_5025Metric
- R24: value 10K -> 470
- R25: value 100K -> 470
- R55: footprint MainBoard:pwr163 -> Eagle_Main:PWR163
- R64, R66: value 10M -> 10M 1%
- R65, R67: value 71K5 -> 71K5 1%
- RN1, RN10, RN11, RN12, RN13, RN14, RN15, RN16, RN17, RN18, RN19, RN2, RN20, RN21, RN22, RN3, RN4, RN5, RN6, RN7, RN8, RN9: footprint MainBoard:R_network_4x1_bourns_CAY16 -> Resistor_SMD:R_Array_Convex_4x0603
- SW1, SW2: footprint MainBoard:Button_SMD_6x3.5x4.3mm -> Button_Switch_SMD:SW_SPST_FSMSM
- TP10: value TS_DIVIDER -> CH4
- TP18: value TS_OVER_60V -> CH4_BF
- TP20: value AIR+_GATE -> AIR+_DELAY
- TP21: value AIR-_GATE -> AIR-_DELAY
- TP24: value SD_OK -> SD_RELAY_D
- TP29, TP30, TP31: footprint MainBoard:TestPoint_GNDedge -> Eagle_Main:TestPoint_GNDedge
- TP4: value FROM_SD -> SD_IN
- TP5: value FROM_TSMS -> SD_END
- TP6: value TO_TSMS -> SD_OUT
- TP7: value BSPD_SIG -> EXT_FAULT
- U1: footprint MainBoard:Tex_DCDC_vertical -> Eagle_Main:Tex_DCDC_vertical_up
- U11: value TS3704IPT -> ADR280ARTZ; footprint Package_SO:TSSOP-14_4.4x5mm_P0.65mm -> Package_TO_SOT_SMD:SOT-23
- U13: value TS3704IPT -> MAX22245; footprint Package_SO:TSSOP-14_4.4x5mm_P0.65mm -> Package_SO:SOIC-8_7.5x5.85mm_P1.27mm
- U15: value CD4082 -> MAX22246; footprint Package_SO:TSSOP-14_4.4x5mm_P0.65mm -> Package_SO:SOIC-8_7.5x5.85mm_P1.27mm
- U16: value ADCMP350 -> ADC124S; footprint Package_TO_SOT_SMD:Analog_KS-4 -> Package_SO:VSSOP-10_3x3mm_P0.5mm
- U27: footprint MainBoard:RFMM -> Eagle_Main:RFMM_0505S
- U4: value MainBoard_AD8244 -> TS3702IPT; footprint Package_SO:MSOP-10_3x3mm_P0.5mm -> Package_SO:TSSOP-8_4.4x3mm_P0.65mm; moved to F.Cu
- U7: value ADCMP354 -> TCMT1103; footprint Package_TO_SOT_SMD:Analog_KS-4 -> Package_SO:SOP-4_4.4x2.6mm_P1.27mm
- Y1: value 26MHz -> 16MHz
- moved TP26 130.2 mm to (249.8, 104.5)
- moved TP25 127.9 mm to (246.8, 104.5)
- moved TP28 120.9 mm to (252.9, 104.5), turned to 0 degrees
- moved RN19 107.2 mm to (124.9, 15.3), turned to 0 degrees
- moved TP18 103.0 mm to (250.7, -18.4)
- moved Q9 94.9 mm to (139.0, -28.2), turned to 0 degrees
- moved R26 92.5 mm to (220.6, 85.0), turned to 0 degrees
- moved R20 91.3 mm to (216.8, 70.2), turned to 90 degrees
- moved Q11 89.5 mm to (131.2, -28.2), turned to 0 degrees
- moved Q10 89.5 mm to (135.1, -28.2), turned to 0 degrees
- moved RN20 86.6 mm to (130.6, -20.9)
- moved TP20 86.4 mm to (251.2, -13.2)
- moved TP21 86.4 mm to (251.2, -15.3)
- moved C34 83.5 mm to (136.5, -4.62)
- moved Q12 83.5 mm to (146.1, -19.1), turned to 0 degrees
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Connections:
- net /AIRs/dissipation renamed Net-(R55-Pad3)
- net /AMS/3V3_FT renamed /MCU/3V3_FT
- net /AMS/BOOT0 renamed /MCU/BOOT0
- net /AMS/CAN_RX renamed /MCU/CAN_RX
- net /AMS/CAN_TX renamed /MCU/CAN_TX
- net /AMS/CARD_OK renamed /MCU/CARD_DET
- net /AMS/CS_CARD renamed /MCU/CS_CARD
- net /AMS/CS_EEPROM renamed /MCU/CS_EEPROM
- net /AMS/FB_FROM_TSMS renamed /MCU/FB_SD_END
- net /AMS/ISO_CAN_RX renamed /MCU/ISO_CAN_RX
- net /AMS/ISO_CAN_TX renamed /MCU/ISO_CAN_TX
- net /AMS/Ip_high renamed /MCU/Ip_high
- net /AMS/Ip_low renamed /MCU/Ip_low
- net /AMS/LED_1 renamed /MCU/LED_1
- net /AMS/LED_2 renamed /MCU/LED_2
- net /AMS/MUX_OUTPUT renamed /MCU/MUX_OUTPUT
- net /AMS/PA15 renamed /MCU/PA15
- net /AMS/PA3 renamed /MCU/PA3
- net /AMS/PA8 renamed /MCU/PA8
- net /AMS/PB1 renamed /MCU/PB1
- net /AMS/PB12 renamed /MCU/PB12
- net /AMS/PB4 renamed /MCU/PB4
- net /AMS/PC0 renamed /MCU/PC0
- net /AMS/PC13 renamed /MCU/PC13
- net /AMS/~HOLD~ renamed /MCU/~HOLD~
- net /AMS/~W~ renamed /MCU/~W~
- net /FROM_SD renamed /SD_IN
- net /FROM_TSMS renamed /SD_END
- net /HIGH_CURRENT renamed /MCU/HIGH_CURRENT
- net /LOW_CURRENT renamed /MCU/LOW_CURRENT
- net /TO_TSMS renamed /SD_OUT
- C17 pad 1: Net-(C17-Pad1) -> /HV/3V3ISO
- C33 pad 1: /NRST_SD -> /SD_RESET
- D11 pad 2: GND -> /AIRs/PRECHARGE_D
- D14 pad 1: Net-(D14-Pad1) -> +5V
- D14 pad 2: GND -> Net-(BZ1-Pad2)
- D15 pad 2: Net-(D15-Pad2) -> /Probing/SD_RELAY_D
- D19 pad 1: Net-(C17-Pad1) -> /AIRs/PRECHARGE_D
- D19 pad 2: /HV/CELLBOARD_5V -> GND
- F3 pad 1: Net-(F3-Pad1) -> /TSAL_12V
- J11 pad 1: /HV/ISO_CANL -> /HV/CAN-
- J11 pad 2: /HV/ISO_CANH -> /HV/CAN+
- J12 pad 3: /AMS/PB7 -> /MCU/PB7
- J17 pad 1: -BATT -> -TS
- J17 pad 2: -TS -> -BATT
- J7 pad 10: Net-(F3-Pad1) -> /EXT_FAULT
- J7 pad 11: GND -> /TSAL
- J7 pad 12: GND -> /TSAL_12V
- J7 pad 4: /NRST_SD -> /SD_RESET
- J7 pad 5: /BMS_LED -> /BMS_COCKPIT
- J7 pad 6: /IMD_LED -> /IMD_COCKPIT
- J7 pad 7: /TSAL -> GND
- J7 pad 8: /CHARGE -> GND
- J7 pad 9: /BSPD_SIG -> /HANDCART_DETECTION
- J8 pad 1: /HV/VS- -> /HV/VS+
- J8 pad 2: /HV/VS+ -> /HV/VS-
- J9 pad 3: /AMS/MOSI_2 -> /MCU/SPI2_MOSI
- J9 pad 5: /AMS/SCK_2 -> /MCU/SPI2_SCK
- J9 pad 7: /AMS/MISO_2 -> /MCU/SPI2_MISO
- JP3 pad 2: /AMS/SCK_2 -> /MCU/SCK_2
- JP7 pad 1: GND -> Net-(J10-Pad3)
- JP7 pad 2: /NRST_SD -> GND
- K1 pad 2: GND -> /AIRs/PRECHARGE_D
- K1 pad 3: Net-(K1-Pad3) -> /AIRs/PRECHARGE_HV_SENSE
- K2 pad 1: Net-(D15-Pad2) -> /Probing/SD_RELAY_D
- Q1 pad 2: +12V -> GND
- Q1 pad 3: Net-(Q1-Pad3) -> Net-(BZ1-Pad2)
- Q10 pad 2: +12V -> Net-(Q10-Pad2)
- Q10 pad 3: Net-(Q1-Pad3) -> Net-(Q10-Pad3)
- Q11 pad 2: +12V -> Net-(Q11-Pad2)
- Q11 pad 3: Net-(Q1-Pad3) -> Net-(Q10-Pad2)
- Q12 pad 2: +12V -> Net-(Q12-Pad2)
- Q12 pad 3: Net-(Q1-Pad3) -> /TSAL
- Q2 pad 2: GND -> Net-(Q13-Pad3)
- Q2 pad 3: Net-(D15-Pad2) -> /Probing/SD_RELAY_D
- Q3 pad 2: GND -> Net-(J6-Pad3)
- Q3 pad 3: Net-(J6-Pad3) -> GND
- Q7 pad 2: GND -> Net-(J10-Pad3)
- Q7 pad 3: Net-(J10-Pad3) -> GND
- Q8 pad 2: +12V -> GND
- Q8 pad 3: /BMS_LED -> /MCU/FAN_PWM
- Q9 pad 2: +12V -> Net-(Q10-Pad3)
- Q9 pad 3: /IMD_LED -> Net-(Q20-Pad2)
- R10 pad 2: /HV/TSV -> Net-(R10-Pad2)
- R16 pad 1: Net-(R16-Pad1) -> +TS
- R16 pad 2: /HV/3V3ISO -> /HV/TS_SENSE
- R18 pad 2: /HV/PackV -> Net-(R18-Pad2)
- R19 pad 1: /HV/~RST~_8902 -> /HV/TS_SENSE
- R19 pad 2: Net-(R16-Pad1) -> -BATT
- R20 pad 1: Net-(D4-Pad1) -> /HV/PRECHARGE_SENSE
- R20 pad 2: /TSAL -> /AIRs/PRECHARGE_HV_SENSE
- R21 pad 1: Net-(R21-Pad1) -> /HV/PRECHARGE_SENSE
- R21 pad 2: /HV/5VISO -> -BATT
- R24 pad 1: +12V -> Net-(R24-Pad1)
- R24 pad 2: /Probing/FB_OVER_60V_12V -> Net-(R24-Pad2)
- R25 pad 1: GND -> Net-(R25-Pad1)
- R25 pad 2: /BSPD_SIG -> Net-(R25-Pad2)
- R26 pad 1: +12V -> /HV/ADC_CH4
- R26 pad 2: /HV/PRECHARGE_STATUS -> Net-(R26-Pad2)
- R36 pad 1: /HV/ISO_CANL -> /HV/CAN+
- R36 pad 2: /HV/ISO_CANH -> /HV/CAN+
- R55 pad 1: Net-(K1-Pad3) -> /AIRs/PRECHARGE_HV_SENSE
- R6 pad 1: +3V3 -> +5V
- R6 pad 2: /AMS/SPI2_MISO -> /MCU/FAN_PWM
- R9 pad 1: /NRST_SD -> /SD_RESET
- RN10 pad 5: /Probing/FB_AIR+_GATE -> /Probing/FB_EXT_LATCHED
- RN10 pad 6: /Probing/FB_AIR- -> /Probing/FB_EXT_LATCHED
- RN10 pad 7: /Probing/FB_AIR+ -> /Probing/FB_EXT_LATCHED
- RN10 pad 8: /Probing/FB_LATCH_BMS -> /Probing/FB_EXT_LATCHED
- RN11 pad 5: /Probing/FB_LATCH_IMD -> /Probing/FB_EXT_LATCHED
- RN11 pad 6: /Probing/FB_BMS_SD -> /Probing/FB_EXT_LATCHED
- RN11 pad 7: /Probing/FB_IMD_SD -> /Probing/FB_EXT_LATCHED
- RN11 pad 8: /Probing/FB_BMS_12V -> /Probing/FB_EXT_LATCHED
- RN12 pad 6: /AMS/TS_ON -> /MCU/TS_ON
- RN12 pad 7: /AMS/BMS_FAULT -> /MCU/BMS_FAULT
- RN12 pad 8: /AMS/ADC_SIN -> /MCU/FAN_PWM_N
- RN13 pad 1: +12V -> +3V3
- RN13 pad 2: +3V3 -> GND
- RN13 pad 3: GND -> Net-(RN13-Pad3)
- RN13 pad 6: /Shutdown/VREF_1.5V -> Net-(RN13-Pad6)
- RN13 pad 8: /HV/PRECHARGE_ON -> /Shutdown/VREF_1.5V
- RN14 pad 1: Net-(RN14-Pad1) -> /MCU/SPI2_MOSI
- RN14 pad 2: /AMS/SPI2_MOSI -> /MCU/SPI2_MISO
- RN14 pad 3: /AMS/SPI2_SCK -> /MCU/SPI2_SCK
- RN14 pad 4: /AMS/SPI2_MISO -> Net-(RN14-Pad4)
- RN14 pad 5: /AMS/MISO_2 -> Net-(RN14-Pad5)
- RN14 pad 6: /AMS/SCK_2 -> /MCU/SPI2_MOSI_
- RN14 pad 7: /AMS/MOSI_2 -> /MCU/SPI2_MISO_
- RN14 pad 8: Net-(RN14-Pad8) -> /MCU/SPI2_SCK_
- RN16 pad 1: GND -> Net-(C37-Pad1)
- RN16 pad 2: Net-(JP4-Pad2) -> GND
- RN16 pad 8: Net-(C37-Pad1) -> Net-(JP4-Pad2)
- RN17 pad 5: /Probing/FB_TS_ON_12V -> /Probing/FB_EXT_LATCHED
- RN17 pad 6: /Probing/FB_BSPD_SIG -> /Probing/FB_EXT_LATCHED
- RN17 pad 7: /Probing/FB_TSAL -> /Probing/FB_EXT_LATCHED
- RN17 pad 8: /Probing/FB_TSAL_OVER60V -> /Probing/FB_EXT_LATCHED
- RN18 pad 5: /AMS/MUX_A0 -> /MCU/MUX_A0
- RN18 pad 6: /AMS/MUX_A1 -> /MCU/MUX_A1
- RN18 pad 7: /AMS/MUX_A3 -> /MCU/MUX_A3
- RN18 pad 8: /AMS/MUX_A2 -> /MCU/MUX_A2
- RN19 pad 1: Net-(RN19-Pad1) -> Net-(Q8-Pad1)
- RN19 pad 2: Net-(RN19-Pad2) -> Net-(Q1-Pad1)
- RN19 pad 7: /AMS/ADC_TX -> /MCU/BUZZER
- RN19 pad 8: /AMS/ADC_RX -> /MCU/FAN_PWM_N
- RN2 pad 1: /AIRs/AIR-_GATE -> /HV/PRECHARGE_STATUS
- RN2 pad 2: +3V3 -> /HV/TS_OVER_60V_STATUS
- RN2 pad 3: /Probing/FB_RELAY_LV_12V -> +3V3
- RN2 pad 4: /IMD_FAULT -> Net-(RN2-Pad4)
- RN2 pad 5: /AMS/FB_IMD_FAULT -> /Probing/FB_EXT_LATCHED
- RN2 pad 6: /AMS/FB_RELAY_LV -> /Probing/FB_EXT_LATCHED
- RN2 pad 7: /Probing/CHECK_MUX -> /Probing/FB_EXT_LATCHED
- RN2 pad 8: /Probing/FB_AIR-_GATE -> /Probing/FB_EXT_LATCHED
- RN20 pad 1: /HV/PRECHARGE_STATUS -> Net-(Q12-Pad1)
- RN20 pad 4: /Probing/FB_OVER_60V_12V -> Net-(Q21-Pad1)
- RN20 pad 5: Net-(Q12-Pad1) -> Net-(Q19-Pad3)
- RN20 pad 6: Net-(Q11-Pad1) -> Net-(Q10-Pad1)
- RN20 pad 7: Net-(Q10-Pad1) -> Net-(Q9-Pad1)
- RN20 pad 8: Net-(Q1-Pad1) -> Net-(Q19-Pad3)
- RN21 pad 1: Net-(Q4-Pad1) -> Net-(RN21-Pad1)
- RN21 pad 2: /Probing/FB_RELAY_LV_12V -> Net-(RN21-Pad2)
- RN21 pad 3: Net-(Q8-Pad1) -> /BMS_COCKPIT
- RN21 pad 4: Net-(Q9-Pad1) -> /IMD_COCKPIT
- RN21 pad 5: /Probing/FB_LATCH_IMD_12V -> Net-(RN21-Pad5)
- RN21 pad 6: /Shutdown/BMS_LATCHED -> Net-(RN21-Pad6)
- RN21 pad 7: Net-(Q2-Pad1) -> Net-(RN21-Pad7)
- RN21 pad 8: Net-(Q1-Pad3) -> Net-(RN21-Pad8)
- RN3 pad 2: /TSAL -> /AIRs/AIR-_GATE
- RN3 pad 3: /Shutdown/BMS_LATCHED -> /AIRs/AIR+_STATUS
- RN3 pad 4: /Probing/FB_LATCH_IMD_12V -> /AIRs/AIR-_STATUS
- RN3 pad 5: /Probing/FB_LATCH_BMS -> /Probing/FB_EXT_LATCHED
- RN3 pad 6: /Probing/FB_AIR+ -> /Probing/FB_EXT_LATCHED
- RN3 pad 7: /Probing/FB_AIR- -> /Probing/FB_EXT_LATCHED
- RN3 pad 8: /Probing/FB_AIR+_GATE -> /Probing/FB_EXT_LATCHED
- RN4 pad 1: /Probing/FB_TS_ON_TO_12V -> /Probing/SD_RELAY_D
- RN4 pad 2: /Shutdown/EN_BMS_SD -> /TSAL
- RN4 pad 3: /Shutdown/EN_IMD_SD -> /EXT_FAULT
- RN4 pad 4: /Shutdown/BMS_FAULT_12V -> /IMD_FAULT
- RN4 pad 5: /Probing/FB_BMS_12V -> /Probing/FB_EXT_LATCHED
- RN4 pad 6: /Probing/FB_IMD_SD -> /Probing/FB_EXT_LATCHED
- RN4 pad 7: /Probing/FB_BMS_SD -> /Probing/FB_EXT_LATCHED
- RN4 pad 8: /Probing/FB_LATCH_IMD -> /Probing/FB_EXT_LATCHED
- RN5 pad 1: /BSPD_SIG -> /Probing/TS_ON
- RN5 pad 2: /AIRs/AIR-_STATUS -> /Probing/IMD_LATCHED
- RN5 pad 3: /AIRs/AIR+_STATUS -> /Probing/BMS_LATCHED
- RN5 pad 4: /Probing/FB_OVER_60V_12V -> /Probing/EXT_LATCHED
- RN5 pad 5: /Probing/FB_TSAL_OVER60V -> /Probing/FB_EXT_LATCHED
- RN5 pad 6: /Probing/FB_TSAL -> /Probing/FB_EXT_LATCHED
- RN5 pad 7: /Probing/FB_BSPD_SIG -> /Probing/FB_EXT_LATCHED
- RN5 pad 8: /Probing/FB_TS_ON_12V -> /Probing/FB_EXT_LATCHED
- RN6 pad 3: /Probing/FB_TO_TSMS -> /Probing/FB_SD_OUT
- RN6 pad 4: /Probing/FB_FROM_SD -> /Probing/FB_SD_IN
- RN7 pad 5: /Probing/FB_AIR-_GATE -> /Probing/FB_EXT_LATCHED
- RN7 pad 6: /Probing/CHECK_MUX -> /Probing/FB_EXT_LATCHED
- RN7 pad 7: /AMS/FB_RELAY_LV -> /Probing/FB_EXT_LATCHED
- RN7 pad 8: /AMS/FB_IMD_FAULT -> /Probing/FB_EXT_LATCHED
- RN8 pad 1: /CHARGE -> /HANDCART_DETECTION
- RN8 pad 3: /BMS_LED -> /IMD_COCKPIT
- RN8 pad 4: /IMD_LED -> /BMS_COCKPIT
- SW2 pad 1: /NRST_SD -> /SD_RESET
- TP10 pad 1: /HV/TS_DIVIDER -> /HV/ADC_CH4
- TP16 pad 1: /AMS/BMS_FAULT -> /MCU/BMS_FAULT
- TP18 pad 1: /Probing/FB_OVER_60V_12V -> Net-(R26-Pad2)
- TP24 pad 1: /Probing/FB_RELAY_LV_12V -> /Probing/SD_RELAY_D
- TP25 pad 1: /Shutdown/BMS_LATCHED -> /Probing/BMS_LATCHED
- TP26 pad 1: /Probing/FB_LATCH_IMD_12V -> /Probing/IMD_LATCHED
- TP27 pad 1: /AMS/TS_ON -> /MCU/TS_ON
- TP28 pad 1: /Probing/FB_TS_ON_TO_12V -> /Probing/TS_ON
- TP7 pad 1: /BSPD_SIG -> /EXT_FAULT
- U11 pad 1: /AIRs/AIR-_GATE -> /HV/5VISO
- U11 pad 2: /AIRs/AIR+_GATE -> /HV/REF_1.2V
- U11 pad 3: +12V -> -BATT
- U12 pad 2: /AMS/MISO_2 -> /MCU/SPI2_MISO
- U12 pad 5: /AMS/MOSI_2 -> /MCU/SPI2_MOSI
- U12 pad 6: /AMS/SCK_2 -> /MCU/SPI2_SCK
- U13 pad 1: /Shutdown/BMS_FAULT_12V -> +3V3
- U13 pad 2: /HV/PRECHARGE_ON -> /HV/ADC_~CS~
- U13 pad 3: +12V -> /HV/ADC_MOSI
- U13 pad 4: +3V3 -> GND
- U13 pad 5: Net-(D14-Pad1) -> -BATT
- U13 pad 6: /Shutdown/VREF_1.5V -> Net-(U13-Pad6)
- U13 pad 7: /AMS/BMS_FAULT -> Net-(U13-Pad7)
- U13 pad 8: /Shutdown/VREF_1.5V -> /HV/3V3ISO
- U14 pad 10: /Probing/FB_LATCH_IMD_12V -> /Probing/IMD_LATCHED
- U14 pad 11: /NRST_SD -> /SD_RESET
- U14 pad 13: Net-(U14-Pad13) -> /Probing/EXT_LATCHED
- U14 pad 3: Net-(U14-Pad3) -> /SD_RESET
- U14 pad 4: Net-(U14-Pad4) -> /EXT_FAULT
- U14 pad 6: /Shutdown/BMS_FAULT_12V -> /Shutdown/BMS_FAULT
- U14 pad 7: /NRST_SD -> /SD_RESET
- U14 pad 9: /Shutdown/BMS_LATCHED -> /Probing/BMS_LATCHED
- U15 pad 1: /HV/PRECHARGE_STATUS -> +3V3
- U15 pad 2: /Probing/FB_OVER_60V_12V -> /HV/ADC_MISO
- U15 pad 3: /HV/PRECHARGE_ON -> /HV/ADC_SCLK
- U15 pad 4: +12V -> GND
- U15 pad 5: +12V -> -BATT
- U15 pad 7: GND -> Net-(U15-Pad7)
- U15 pad 8: Net-(U15-Pad8) -> /HV/3V3ISO
- U16 pad 1: /HV/TS_DIVIDER -> Net-(U13-Pad7)
- U16 pad 2: -BATT -> /HV/3V3ISO
- U16 pad 3: /HV/PROMINENT- -> -BATT
- U16 pad 4: Net-(C17-Pad1) -> /HV/ADC_CH4
- U24 pad 1: /HV/PackV -> Net-(R18-Pad2)
- U24 pad 2: /HV/PackV -> Net-(R42-Pad2)
- U24 pad 6: /HV/TSV -> Net-(R41-Pad2)
- U24 pad 7: /HV/TSV -> Net-(R10-Pad2)
- U30 pad 6: /HV/ISO_CANL -> /HV/CAN+
- U30 pad 7: /HV/ISO_CANH -> /HV/CAN+
- U4 pad 1: /Shutdown/BMS_LATCHED -> Net-(RN25-Pad5)
- U4 pad 2: /Shutdown/EN_BMS_SD -> Net-(JP5-Pad2)
- U4 pad 3: +12V -> Net-(C37-Pad1)
- U4 pad 4: /Shutdown/EN_IMD_SD -> GND
- U4 pad 5: /Probing/FB_LATCH_IMD_12V -> Net-(C31-Pad1)
- U4 pad 6: /Probing/FB_LATCH_IMD_12V -> +3V3
- U4 pad 7: /IMD_LED -> Net-(RN25-Pad7)
- U4 pad 8: GND -> +12V
- U6 pad 2: Net-(R17-Pad2) -> Net-(R4-Pad2)
- U6 pad 6: Net-(R22-Pad2) -> Net-(R37-Pad2)
- U7 pad 1: /HV/TS_DIVIDER -> /HV/5VISO
- U7 pad 2: -BATT -> Net-(R24-Pad1)
- U7 pad 3: Net-(U19-Pad2) -> /HV/TS_OVER_60V_STATUS
- U7 pad 4: /HV/5VISO -> +12V
- U8 pad 10: /AMS/MUX_A0 -> /MCU/MUX_A0
- U8 pad 11: /AMS/MUX_A1 -> /MCU/MUX_A1
- U8 pad 13: /AMS/MUX_A3 -> /MCU/MUX_A3
- U8 pad 14: /AMS/MUX_A2 -> /MCU/MUX_A2
- U8 pad 16: /Probing/FB_TO_TSMS -> /Probing/FB_EXT_LATCHED
- U8 pad 17: /Probing/FB_FROM_SD -> /Probing/FB_EXT_LATCHED
- U8 pad 18: /Probing/CHECK_MUX -> /Probing/FB_EXT_LATCHED
- U8 pad 19: /Probing/FB_AIR-_GATE -> /Probing/FB_EXT_LATCHED
- U8 pad 2: /Probing/FB_BMS_12V -> /Probing/FB_EXT_LATCHED
- U8 pad 20: /Probing/FB_LATCH_BMS -> /Probing/FB_EXT_LATCHED
- U8 pad 21: /Probing/FB_AIR+ -> /Probing/FB_EXT_LATCHED
- U8 pad 22: /Probing/FB_AIR- -> /Probing/FB_EXT_LATCHED
- U8 pad 23: /Probing/FB_AIR+_GATE -> /Probing/FB_EXT_LATCHED
- U8 pad 3: /Probing/FB_IMD_SD -> /Probing/FB_EXT_LATCHED
- U8 pad 4: /Probing/FB_BMS_SD -> /Probing/FB_EXT_LATCHED
- U8 pad 5: /Probing/FB_LATCH_IMD -> /Probing/FB_EXT_LATCHED
- U8 pad 6: /Probing/FB_TSAL_OVER60V -> /Probing/FB_EXT_LATCHED
- U8 pad 7: /Probing/FB_TSAL -> /Probing/FB_EXT_LATCHED
- U8 pad 8: /Probing/FB_BSPD_SIG -> /Probing/FB_EXT_LATCHED
- U8 pad 9: /Probing/FB_TS_ON_12V -> /Probing/FB_EXT_LATCHED
- U9 pad 15: /AMS/FB_RELAY_LV -> /MCU/FB_SD_RELAY_D
- U9 pad 16: /AMS/FB_IMD_FAULT -> /MCU/FB_IMD_FAULT
- U9 pad 21: /AMS/MUX_A0 -> /MCU/SPI1_SCK_
- U9 pad 22: /AMS/MUX_A1 -> /MCU/SPI1_MISO_
- U9 pad 23: /AMS/MUX_A2 -> /MCU/SPI1_MOSI_
- U9 pad 24: /AMS/MUX_A3 -> /MCU/CS_ADC_
- U9 pad 25: /AMS/ADC_RX -> Net-(U9-Pad25)
- U9 pad 26: /AMS/ADC_SIN -> Net-(U9-Pad26)
- U9 pad 29: /AMS/ADC_TX -> Net-(U9-Pad29)
- U9 pad 34: /AMS/SPI2_SCK -> /MCU/SPI2_SCK_
- U9 pad 35: /AMS/SPI2_MISO -> /MCU/SPI2_MISO_
- U9 pad 36: /AMS/SPI2_MOSI -> /MCU/SPI2_MOSI_
- U9 pad 51: /AMS/BMS_FAULT -> /MCU/BMS_FAULT
- U9 pad 52: /AMS/TS_ON -> /MCU/TS_ON
- U9 pad 59: /AMS/PB7 -> /MCU/FAN_PWM_N
- U9 pad 9: /CHARGE -> /HANDCART
Routing:
- net +12V: track 449.1 -> 193.7 mm, vias 14 -> 3
- net /Probing/FB_EXT_LATCHED: track 0.00 -> 186.2 mm, vias 0 -> 28
- net /Probing/FB_OVER_60V_12V: track 111.4 -> 0.00 mm, vias 6 -> 0
- net /TSAL: track 84.8 -> 0.00 mm, vias 7 -> 0
- net /AMS/ADC_SIN: track 83.5 -> 0.00 mm, vias 3 -> 0
- net /BSPD_SIG: track 80.7 -> 0.00 mm, vias 6 -> 0
- net /Shutdown/BMS_LATCHED: track 75.2 -> 0.00 mm, vias 5 -> 0
- net Net-(U9-Pad26): track 0.00 -> 74.9 mm, vias 0 -> 3
- net /Shutdown/BMS_FAULT_12V: track 73.5 -> 0.00 mm, vias 6 -> 0
- net /Probing/FB_LATCH_IMD_12V: track 71.2 -> 0.00 mm, vias 9 -> 0
- net /Probing/FB_RELAY_LV_12V: track 66.8 -> 0.00 mm, vias 5 -> 0
- net /Probing/FB_TS_ON_TO_12V: track 65.6 -> 0.00 mm, vias 5 -> 0
- net /IMD_FAULT: track 99.4 -> 35.1 mm, vias 4 -> 0
- net Net-(Q2-Pad1): track 62.4 -> 0.00 mm, vias 4 -> 0
- net /AIRs/AIR+_STATUS: track 61.5 -> 0.00 mm, vias 4 -> 0
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- added copper zone on B.Cu, net /AIRs/dissipation
- added copper zone on F.Cu, net /AIRs/dissipation
- removed copper zone on B.Cu, net -BATT
- removed copper zone on F.Cu, net -BATT
- removed copper zone on B.Cu, net Net-(R55-Pad3)
- removed copper zone on F.Cu, net Net-(R55-Pad3)
Other:
- net class RELAY removed
- net class SD_AIR added: clearance 0.5, trace_width 0.25, via_dia 0.55, via_drill 0.25
- board text removed: "+BATT"
- board text removed: "+TS"
- board text removed: "-BATT"
- board text removed: "-TS"
- board text removed: "GLVS"
- board text removed: "HV ISOLATED ADC"
- board text removed: "OVER 60V DETECTION + PROMINENT"
- board text removed: "PROMINET"
