File: mainboard/Probing.sch (KiCad schematic (older format))
At the start: 19 parts, among them U8 CD74HC4067SM

Commit message: Correction almost finished, Started layouting
Parts:
- RN10, RN11, RN17, RN18, RN2, RN3, RN4, RN5, RN6, RN7: footprint MainBoard:R_network_4x1_bourns_CAY16 -> Resistor_SMD:R_Array_Convex_4x0603
Connections:
- net FB_AIR+ is gone; now on net FB_EXT_LATCHED: RN10.7 (R2.2), RN3.6 (R3.2), U8.21 (I10)
- net FB_AIR+_GATE is gone; now on net FB_EXT_LATCHED: RN10.5 (R4.2), RN3.8 (R1.2), U8.23 (I8)
- net FB_AIR- is gone; now on net FB_EXT_LATCHED: RN10.6 (R3.2), RN3.7 (R2.2), U8.22 (I9)
- net FB_AIR-_GATE is gone; now on net FB_EXT_LATCHED: RN2.8 (R1.2), RN7.5 (R4.2), U8.19 (I12)
- net FB_BMS_12V is gone; now on net FB_EXT_LATCHED: RN11.8 (R1.2), RN4.5 (R4.2), U8.2 (I7)
- net FB_BMS_SD is gone; now on net FB_EXT_LATCHED: RN11.6 (R3.2), RN4.7 (R2.2), U8.4 (I5)
- net FB_BSPD_SIG is gone; now on net FB_EXT_LATCHED: RN17.6 (R3.2), RN5.7 (R2.2), U8.8 (I1)
- net FB_IMD_FAULT is gone; now on net FB_EXT_LATCHED: RN2.5 (R4.2), RN7.8 (R1.2)
- net FB_IMD_SD is gone; now on net FB_EXT_LATCHED: RN11.7 (R2.2), RN4.6 (R3.2), U8.3 (I6)
- net FB_LATCH_BMS is gone; now on net FB_EXT_LATCHED: RN10.8 (R1.2), RN3.5 (R4.2), U8.20 (I11)
- net FB_LATCH_IMD is gone; now on net FB_EXT_LATCHED: RN11.5 (R4.2), RN4.8 (R1.2), U8.5 (I4)
- net FB_RELAY_LV is gone; now on net FB_EXT_LATCHED: RN2.6 (R3.2), RN7.7 (R2.2)
- net FB_RELAY_LV_12V is gone; now on net +3V3: RN2.3 (R3.1)
- net FB_TSAL is gone; now on net FB_EXT_LATCHED: RN17.7 (R2.2), RN5.6 (R3.2), U8.7 (I2)
- net FB_TSAL_OVER60V is gone; now on net FB_EXT_LATCHED: RN17.8 (R1.2), RN5.5 (R4.2), U8.6 (I3)
- net FB_TS_ON_12V is gone; now on net FB_EXT_LATCHED: RN17.5 (R4.2), RN5.8 (R1.2), U8.9 (I0)
- net +3V3: no longer RN2.2 (R2.1)
- net CHECK_MUX renamed FB_EXT_LATCHED
- net FB_EXT_LATCHED: now also U8.16 (I15), U8.17 (I14)
- net FB_AIR+_12V renamed BMS_LATCHED
- net FB_AIR+_GATE_12V renamed AIR+_GATE
- net FB_AIR-_12V renamed IMD_LATCHED
- net FB_AIR-_GATE_12V renamed PRECHARGE_STATUS
- net FB_BMS_SD_12V renamed TSAL
- net FB_BMS_TO_12V renamed IMD_FAULT
- net FB_BSPD_SIG_12V renamed TS_ON
- net FB_FROM_SD renamed FB_SD_IN
- net FB_SD_IN: no longer U8.17 (I14)
- net FB_FROM_TSMS renamed FB_SD_END
- net FB_IMD_FAULT_12V: no longer names the net of RN2.4 (R4.1)
- net FB_IMD_SD_12V renamed EXT_FAULT
- net FB_LATCH_BMS_12V renamed AIR+_STATUS
- net FB_LATCH_IMD_12V renamed AIR-_STATUS
- net FB_OVER_60V_12V renamed EXT_LATCHED
- net FB_TO_TSMS renamed FB_SD_OUT
- net FB_SD_OUT: no longer U8.16 (I15)
- net FB_TSAL_12V renamed AIR-_GATE
- net FB_TS_ON_TO_12V renamed SD_RELAY_D
- net FROM_SD renamed SD_IN
- net FROM_TSMS renamed SD_END
- net TO_TSMS renamed SD_OUT
- new net TS_OVER_60V_STATUS: RN2.2 (R2.1)
Other:
- note added: "I=12V/430K=2.79*10^(-5)A\nR=330K-->0.26mW\nR=100K-->0.078mW"
- note added: "RECHECK ALL OF THE FEEDBACK NAMES"
- note added: "Shutdown check"
- note removed: "I=12V/430K=2.79*10^(-5)\nR=330K-->0.26mW\nR=100K-->0.078mW"
- note removed: "current into R14-R16\nif Vsd=12V--->9uA\nif Vsd=55V--->52uA"
- moved on the sheet: C18, D5, D6, D7, R13, R14, R15, TP17
